File: Eagle/UCirKitBreadboard/UCirKitBreadboard.brd (EAGLE design)
At the start: 73.6 x 100 mm, 160 parts

Commit message: breadboard version
Parts:
- removed JP101, JP102, JP103, JP104, JP105, JP106, JP107, JP108, JP109, JP110, JP111, JP112, JP113, JP114, JP115, JP116, JP117, JP118, JP119, JP120, JP121, JP122, JP123, JP124, JP125, JP126, JP127, JP128, JP129, JP130, JP131, JP132, JP133, JP134, JP135, JP136, JP137, JP138, JP139, JP140, JP141, JP142, JP143, JP144, JP145, JP146, JP147, JP148, JP149, JP150, JP151, JP152, JP153, JP154, JP155, JP156, JP157, JP158, JP159, JP160: (no value), SparkFun-Connectors:1X05-1.27MM
- removed JP21, JP22, JP23, JP24, JP25, JP26, JP27, JP28, JP29, JP30, JP31, JP32, JP33, JP34, JP35, JP36, JP37, JP38, JP39, JP40: (no value), SparkFun-Connectors:1X15
- moved JP92 88.5 mm to (18.4, 93.3), turned to 0 degrees
- moved JP91 86.7 mm to (12.1, 93.3), turned to 0 degrees
- moved JP65 84.9 mm to (48.3, 87.0), turned to 270 degrees
- moved JP77 80.4 mm to (50.2, 87.0), turned to 270 degrees
- moved JP66 76.5 mm to (48.3, 80.6), turned to 270 degrees
- moved JP90 76.3 mm to (18.4, 91.4), turned to 0 degrees
- moved JP97 76.3 mm to (12.1, 7.62), turned to 0 degrees
- moved JP89 75.5 mm to (12.1, 91.4), turned to 0 degrees
- moved JP78 73.3 mm to (50.2, 80.6), turned to 270 degrees
- moved JP67 68.3 mm to (48.3, 74.3), turned to 270 degrees
- moved JP98 67.4 mm to (18.4, 7.62), turned to 0 degrees
- moved JP79 66.7 mm to (50.2, 74.3), turned to 270 degrees
- moved JP80 60.7 mm to (50.2, 67.9), turned to 270 degrees
- moved JP68 60.3 mm to (48.3, 67.9), turned to 270 degrees
- moved JP99 53.3 mm to (32.4, 7.62), turned to 0 degrees
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Connections:
- new net N$215: JP15.11
- new net N$216: JP15.10
- new net N$217: JP15.9
- new net N$218: JP15.8
- new net N$219: JP15.7
- new net N$220: JP15.6
- new net N$221: JP15.5
- new net N$222: JP15.4
- new net N$223: JP15.3
- new net N$224: JP15.2
- new net N$225: JP15.1
- new net N$226: JP16.15
- new net N$227: JP16.14
- new net N$228: JP16.13
- new net N$229: JP16.12
- new net N$230: JP16.11
- new net N$231: JP16.10
- new net N$232: JP16.9
- new net N$233: JP16.8
- new net N$234: JP16.7
- new net N$235: JP16.6
- new net N$236: JP16.5
- new net N$237: JP16.4
- new net N$238: JP16.3
- new net N$239: JP16.2
- new net N$240: JP16.1
- new net N$241: JP17.15
- new net N$242: JP17.14
- new net N$243: JP17.13
- new net N$244: JP17.12
- new net N$245: JP17.11
- new net N$246: JP17.10
- new net N$247: JP17.9
- new net N$248: JP17.8
- new net N$249: JP17.7
- new net N$250: JP17.6
- new net N$251: JP17.5
- new net N$252: JP17.4
- new net N$253: JP17.3
- new net N$254: JP17.2
- new net N$255: JP17.1
- new net N$256: JP18.15
- new net N$257: JP18.14
- new net N$258: JP18.13
- new net N$259: JP18.12
- new net N$260: JP18.11
- new net N$261: JP18.10
- new net N$262: JP18.9
- new net N$263: JP18.8
- new net N$264: JP18.7
- new net N$265: JP18.6
- new net N$266: JP18.5
- new net N$267: JP18.4
- new net N$268: JP18.3
- new net N$269: JP18.2
- new net N$270: JP18.1
- new net N$271: JP19.15
- new net N$272: JP19.14
- new net N$273: JP19.13
- new net N$274: JP19.12
- new net N$275: JP19.11
- new net N$276: JP19.10
- new net N$277: JP19.9
- new net N$278: JP19.8
- new net N$279: JP19.7
- new net N$280: JP19.6
- new net N$281: JP19.5
- new net N$282: JP19.4
- new net N$283: JP19.3
- new net N$284: JP19.2
- new net N$285: JP19.1
- new net N$286: JP20.15
- new net N$287: JP20.14
- new net N$288: JP20.13
- new net N$289: JP20.12
- new net N$290: JP20.11
- new net N$291: JP20.10
- new net N$292: JP20.9
- new net N$293: JP20.8
- new net N$294: JP20.7
- new net N$295: JP20.6
- new net N$296: JP20.5
- new net N$297: JP20.4
- new net N$298: JP20.3
- new net N$299: JP20.2
- new net N$300: JP20.1
- new net N$601: JP41.5
- new net N$602: JP41.4
- new net N$603: JP41.3
- new net N$604: JP41.2
- new net N$605: JP41.1
- new net N$606: JP42.5
- new net N$607: JP42.4
- new net N$608: JP42.3
- new net N$609: JP42.2
- new net N$610: JP42.1
- new net N$611: JP43.5
- new net N$612: JP43.4
- new net N$613: JP43.3
- new net N$614: JP43.2
- new net N$615: JP43.1
- new net N$616: JP44.5
- new net N$617: JP44.4
- new net N$618: JP44.3
- new net N$619: JP44.2
- new net N$620: JP44.1
- new net N$621: JP45.5
- new net N$622: JP45.4
- new net N$623: JP45.3
- new net N$624: JP45.2
- new net N$625: JP45.1
- new net N$626: JP46.5
- new net N$627: JP46.4
- new net N$628: JP46.3
- new net N$629: JP46.2
- new net N$630: JP46.1
- new net N$631: JP47.5
- new net N$632: JP47.4
- new net N$633: JP47.3
- new net N$634: JP47.2
- new net N$635: JP47.1
- new net N$636: JP48.5
- new net N$637: JP48.4
- new net N$638: JP48.3
- new net N$639: JP48.2
- new net N$640: JP48.1
- new net N$641: JP49.5
- new net N$642: JP49.4
- new net N$643: JP49.3
- new net N$644: JP49.2
- new net N$645: JP49.1
- new net N$646: JP50.5
- new net N$647: JP50.4
- new net N$648: JP50.3
- new net N$649: JP50.2
- new net N$650: JP50.1
- new net N$651: JP51.5
- new net N$652: JP51.4
- new net N$653: JP51.3
- new net N$654: JP51.2
- new net N$655: JP51.1
- new net N$656: JP52.5
- new net N$657: JP52.4
- new net N$658: JP52.3
- new net N$659: JP52.2
- new net N$660: JP52.1
- new net N$661: JP53.5
- new net N$662: JP53.4
- new net N$663: JP53.3
- new net N$664: JP53.2
- new net N$665: JP53.1
- new net N$666: JP54.5
- new net N$667: JP54.4
- new net N$668: JP54.3
- new net N$669: JP54.2
- new net N$670: JP54.1
- new net N$671: JP55.5
- new net N$672: JP55.4
- new net N$673: JP55.3
- new net N$674: JP55.2
- new net N$675: JP55.1
- new net N$676: JP56.5
- new net N$677: JP56.4
- new net N$678: JP56.3
- new net N$679: JP56.2
- new net N$680: JP56.1
- new net N$681: JP57.5
- new net N$682: JP57.4
- new net N$683: JP57.3
- new net N$684: JP57.2
- new net N$685: JP57.1
- new net N$686: JP58.5
- new net N$687: JP58.4
- new net N$688: JP58.3
- new net N$689: JP58.2
- new net N$690: JP58.1
- new net N$691: JP59.5
- new net N$692: JP59.4
- new net N$693: JP59.3
- new net N$694: JP59.2
- new net N$695: JP59.1
- new net N$696: JP60.5
- new net N$697: JP60.4
- new net N$698: JP60.3
- new net N$699: JP60.2
- new net N$700: JP60.1
- new net N$701: JP61.5
- new net N$702: JP61.4
- new net N$703: JP61.3
- new net N$704: JP61.2
- new net N$705: JP61.1
- new net N$706: JP62.5
- new net N$707: JP62.4
- new net N$708: JP62.3
- new net N$709: JP62.2
- new net N$710: JP62.1
- new net N$711: JP63.5
- new net N$712: JP63.4
- new net N$713: JP63.3
- new net N$714: JP63.2
- new net N$715: JP63.1
- new net N$716: JP64.5
- new net N$717: JP64.4
- new net N$718: JP64.3
- new net N$719: JP64.2
- new net N$720: JP64.1
- new net N$721: JP65.5
- new net N$722: JP65.4
- new net N$723: JP65.3
- new net N$724: JP65.2
- new net N$725: JP65.1
- new net N$726: JP66.5
- new net N$727: JP66.4
- new net N$728: JP66.3
- new net N$729: JP66.2
- new net N$730: JP66.1
- new net N$731: JP67.5
- new net N$732: JP67.4
- new net N$733: JP67.3
- new net N$734: JP67.2
- new net N$735: JP67.1
- new net N$736: JP68.5
- new net N$737: JP68.4
- new net N$738: JP68.3
- new net N$739: JP68.2
- new net N$740: JP68.1
- new net N$741: JP69.5
- new net N$742: JP69.4
- new net N$743: JP69.3
- new net N$744: JP69.2
- new net N$745: JP69.1
- new net N$746: JP70.5
- new net N$747: JP70.4
- new net N$748: JP70.3
- new net N$749: JP70.2
- new net N$750: JP70.1
- new net N$751: JP71.5
- new net N$752: JP71.4
- new net N$753: JP71.3
- new net N$754: JP71.2
- new net N$755: JP71.1
- new net N$756: JP72.5
- new net N$757: JP72.4
- new net N$758: JP72.3
- new net N$759: JP72.2
- new net N$760: JP72.1
- new net N$761: JP73.5
- new net N$762: JP73.4
- new net N$763: JP73.3
- new net N$764: JP73.2
- new net N$765: JP73.1
- new net N$766: JP74.5
- new net N$767: JP74.4
- new net N$768: JP74.3
- new net N$769: JP74.2
- new net N$770: JP74.1
- new net N$771: JP75.5
- new net N$772: JP75.4
- new net N$773: JP75.3
- new net N$774: JP75.2
- new net N$775: JP75.1
- new net N$776: JP76.5
- new net N$777: JP76.4
- new net N$778: JP76.3
- new net N$779: JP76.2
- new net N$780: JP76.1
- new net N$781: JP77.5
- new net N$782: JP77.4
- new net N$783: JP77.3
- new net N$784: JP77.2
- new net N$785: JP77.1
- new net N$786: JP78.5
- new net N$787: JP78.4
- new net N$788: JP78.3
- new net N$789: JP78.2
- new net N$790: JP78.1
- new net N$791: JP79.5
- new net N$792: JP79.4
- new net N$793: JP79.3
- new net N$794: JP79.2
- new net N$795: JP79.1
- new net N$796: JP80.5
- new net N$797: JP80.4
- new net N$798: JP80.3
- new net N$799: JP80.2
- new net N$800: JP80.1
- new net N$801: JP81.5
- new net N$802: JP81.4
- new net N$803: JP81.3
- new net N$804: JP81.2
- new net N$805: JP81.1
- new net N$806: JP82.5
- new net N$807: JP82.4
- new net N$808: JP82.3
- new net N$809: JP82.2
- new net N$810: JP82.1
- new net N$811: JP83.5
- new net N$812: JP83.4
- new net N$813: JP83.3
- new net N$814: JP83.2
- new net N$815: JP83.1
- new net N$816: JP84.5
- new net N$817: JP84.4
- new net N$818: JP84.3
- new net N$819: JP84.2
- new net N$820: JP84.1
- new net N$821: JP85.5
- new net N$822: JP85.4
- new net N$823: JP85.3
- new net N$824: JP85.2
- new net N$825: JP85.1
- new net N$826: JP86.5
- new net N$827: JP86.4
- new net N$828: JP86.3
- new net N$829: JP86.2
- new net N$830: JP86.1
- new net N$831: JP87.5
- new net N$832: JP87.4
- new net N$833: JP87.3
- new net N$834: JP87.2
- new net N$835: JP87.1
- new net N$836: JP88.5
- new net N$837: JP88.4
- new net N$838: JP88.3
- new net N$839: JP88.2
- new net N$840: JP88.1
- new net N$841: JP89.5
- new net N$842: JP89.4
- new net N$843: JP89.3
- new net N$844: JP89.2
- new net N$845: JP89.1
- new net N$846: JP90.5
- new net N$847: JP90.4
- new net N$848: JP90.3
- new net N$849: JP90.2
- new net N$850: JP90.1
- new net N$851: JP91.5
- new net N$852: JP91.4
- new net N$853: JP91.3
- new net N$854: JP91.2
- new net N$855: JP91.1
- new net N$856: JP92.5
- new net N$857: JP92.4
- new net N$858: JP92.3
- new net N$859: JP92.2
- new net N$860: JP92.1
- new net N$861: JP93.5
- new net N$862: JP93.4
- new net N$863: JP93.3
- new net N$864: JP93.2
- new net N$865: JP93.1
- new net N$866: JP94.5
- new net N$867: JP94.4
- new net N$868: JP94.3
- new net N$869: JP94.2
- new net N$870: JP94.1
- new net N$871: JP95.5
- new net N$872: JP95.4
- new net N$873: JP95.3
- new net N$874: JP95.2
- new net N$875: JP95.1
- new net N$876: JP96.5
- new net N$877: JP96.4
- new net N$878: JP96.3
- new net N$879: JP96.2
- new net N$880: JP96.1
- new net N$881: JP97.5
- new net N$882: JP97.4
- new net N$883: JP97.3
- new net N$884: JP97.2
- new net N$885: JP97.1
- new net N$886: JP98.5
- new net N$887: JP98.4
- new net N$888: JP98.3
- new net N$889: JP98.2
- new net N$890: JP98.1
- new net N$891: JP99.5
- new net N$892: JP99.4
- new net N$893: JP99.3
- new net N$894: JP99.2
- new net N$895: JP99.1
- new net N$896: JP100.5
- new net N$897: JP100.4
- new net N$898: JP100.3
- new net N$899: JP100.2
- new net N$900: JP100.1
Other:
- board size 73.6 x 100 mm -> 58.4 x 100 mm
