File: Eagle/UCirKitBreadboard/Test.sch (EAGLE design)
At the start: 80 parts

Commit message: almost done version board
Connections:
- removed net N$717: JP64.4
- new net NEW_300: JP13.15, JP64.4
Changed lines of the file:
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@@
 <?xml version="1.0" encoding="utf-8"?>
 <!DOCTYPE eagle SYSTEM "eagle.dtd">
-<eagle version="6.5.0">
+<eagle version="7.3.0">
 <drawing>
 <settings>
@@
 <pinref part="JP54" gate="G$1" pin="5"/>
 <wire x1="142.24" y1="-33.02" x2="160.02" y2="-33.02" width="0.1524" layer="91"/>
+<label x="142.24" y="-33.02" size="1.778" layer="95"/>
 </segment>
 </net>
@@
 <pinref part="JP52" gate="G$1" pin="3"/>
 <wire x1="111.76" y1="-55.88" x2="129.54" y2="-55.88" width="0.1524" layer="91"/>
+<label x="111.76" y="-55.88" size="1.778" layer="95"/>
 </segment>
 </net>
@@
 <pinref part="JP52" gate="G$1" pin="5"/>
 <wire x1="111.76" y1="-50.8" x2="129.54" y2="-50.8" width="0.1524" layer="91"/>
+<label x="111.76" y="-50.8" size="1.778" layer="95"/>
 </segment>
 </net>
@@
 <pinref part="JP52" gate="G$1" pin="1"/>
 <wire x1="111.76" y1="-60.96" x2="129.54" y2="-60.96" width="0.1524" layer="91"/>
+<label x="111.76" y="-60.96" size="1.778" layer="95"/>
 </segment>
 </net>
@@
 <pinref part="JP52" gate="G$1" pin="2"/>
 <wire x1="111.76" y1="-58.42" x2="129.54" y2="-58.42" width="0.1524" layer="91"/>
+<label x="111.76" y="-58.42" size="1.778" layer="95"/>
 </segment>
 </net>
@@
 <pinref part="JP52" gate="G$1" pin="4"/>
 <wire x1="111.76" y1="-53.34" x2="129.54" y2="-53.34" width="0.1524" layer="91"/>
+<label x="111.76" y="-53.34" size="1.778" layer="95"/>
 </segment>
 </net>
@@
 <pinref part="JP62" gate="G$1" pin="3"/>
 <wire x1="241.3" y1="-20.32" x2="259.08" y2="-20.32" width="0.1524" layer="91"/>
+<label x="241.3" y="-20.32" size="1.778" layer="95"/>
 </segment>
 </net>
@@
 <pinref part="JP62" gate="G$1" pin="5"/>
 <wire x1="241.3" y1="-15.24" x2="259.08" y2="-15.24" width="0.1524" layer="91"/>
+<label x="241.3" y="-15.24" size="1.778" layer="95"/>
 </segment>
 </net>
@@
 <pinref part="JP64" gate="G$1" pin="3"/>
 <wire x1="241.3" y1="-55.88" x2="259.08" y2="-55.88" width="0.1524" layer="91"/>
-</segment>
-</net>
-<net name="N$195" class="0">
-<segment>
-<wire x1="403.86" y1="121.92" x2="424.18" y2="121.92" width="0.1524" layer="91"/>
+<label x="241.3" y="-55.88" size="1.778" layer="95"/>
 </segment>
 </net>
@@
 <pinref part="JP64" gate="G$1" pin="5"/>
 <wire x1="241.3" y1="-50.8" x2="259.08" y2="-50.8" width="0.1524" layer="91"/>
+<label x="241.3" y="-50.8" size="1.778" layer="95"/>
 </segment>
 </net>
@@
 <pinref part="JP64" gate="G$1" pin="2"/>
 <wire x1="241.3" y1="-58.42" x2="259.08" y2="-58.42" width="0.1524" layer="91"/>
+<label x="241.3" y="-58.42" size="1.778" layer="95"/>
 </segment>
 </net>
@@
 <pinref part="JP64" gate="G$1" pin="1"/>
 <wire x1="241.3" y1="-60.96" x2="259.08" y2="-60.96" width="0.1524" layer="91"/>
+<label x="241.3" y="-60.96" size="1.778" layer="95"/>
 </segment>
 </net>
@@
 <pinref part="JP62" gate="G$1" pin="4"/>
 <wire x1="241.3" y1="-17.78" x2="259.08" y2="-17.78" width="0.1524" layer="91"/>
+<label x="241.3" y="-17.78" size="1.778" layer="95"/>
 </segment>
 </net>
@@
 <pinref part="JP62" gate="G$1" pin="2"/>
 <wire x1="241.3" y1="-22.86" x2="259.08" y2="-22.86" width="0.1524" layer="91"/>
+<label x="241.3" y="-22.86" size="1.778" layer="95"/>
 </segment>
 </net>
@@
 <pinref part="JP62" gate="G$1" pin="1"/>
 <wire x1="241.3" y1="-25.4" x2="259.08" y2="-25.4" width="0.1524" layer="91"/>
+<label x="241.3" y="-25.4" size="1.778" layer="95"/>
 </segment>
 </net>
@@
 </segment>
 </net>
-<net name="N$717" class="0">
+<net name="NEW_300" class="0">
+<segment>
+<pinref part="JP13" gate="G$1" pin="15"/>
+<wire x1="406.4" y1="121.92" x2="424.18" y2="121.92" width="0.1524" layer="91"/>
+</segment>
 <segment>
 <pinref part="JP64" gate="G$1" pin="4"/>
 <wire x1="241.3" y1="-53.34" x2="259.08" y2="-53.34" width="0.1524" layer="91"/>
+<label x="241.3" y="-53.34" size="1.778" layer="95"/>
 </segment>
 </net>
