File: Eagle/UCirKit30x10Spacing-0805/UCirKit30x20-0721.brd (EAGLE design)
At the start: 132.1 x 68.2 mm, 80 parts

Commit message: RenameAllNetToClean.ulp script uploaded
Connections:
- net N$10 renamed CLEAN346
- net N$11 renamed CLEAN345
- net N$12 renamed CLEAN354
- net N$13 renamed CLEAN353
- net N$14 renamed CLEAN352
- net N$15 renamed CLEAN351
- net N$16 renamed CLEAN350
- net N$17 renamed CLEAN494
- net N$18 renamed CLEAN493
- net N$19 renamed CLEAN492
- net N$2 renamed CLEAN344
- net N$20 renamed CLEAN491
- net N$21 renamed CLEAN490
- net N$22 renamed CLEAN499
- net N$23 renamed CLEAN498
- net N$24 renamed CLEAN497
- net N$25 renamed CLEAN496
- net N$26 renamed CLEAN495
- net N$27 renamed CLEAN504
- net N$28 renamed CLEAN503
- net N$29 renamed CLEAN502
- net N$3 renamed CLEAN343
- net N$30 renamed CLEAN501
- net N$31 renamed CLEAN500
- net N$4 renamed CLEAN342
- net N$5 renamed CLEAN341
- net N$6 renamed CLEAN340
- net N$7 renamed CLEAN349
- net N$8 renamed CLEAN348
- net N$9 renamed CLEAN347
- net NEW_100 renamed CLEAN132
- net NEW_101 renamed CLEAN131
- net NEW_102 renamed CLEAN133
- net NEW_103 renamed CLEAN134
- net NEW_105 renamed CLEAN98
- net NEW_11 renamed CLEAN28
- net NEW_110 renamed CLEAN97
- net NEW_111 renamed CLEAN101
- net NEW_115 renamed CLEAN470
- net NEW_116 renamed CLEAN471
- net NEW_117 renamed CLEAN472
- net NEW_12 renamed CLEAN14
- net NEW_120 renamed CLEAN465
- net NEW_121 renamed CLEAN466
- net NEW_130 renamed CLEAN56
- net NEW_131 renamed CLEAN54
- net NEW_132 renamed CLEAN55
- net NEW_133 renamed CLEAN57
- net NEW_135 renamed CLEAN111
- net NEW_14 renamed CLEAN27
- net NEW_140 renamed CLEAN113
- net NEW_141 renamed CLEAN114
- net NEW_146 renamed CLEAN481
- net NEW_147 renamed CLEAN482
- net NEW_148 renamed CLEAN483
- net NEW_149 renamed CLEAN484
- net NEW_15 renamed CLEAN58
- net NEW_152 renamed CLEAN477
- net NEW_155 renamed CLEAN123
- net NEW_156 renamed CLEAN124
- net NEW_157 renamed CLEAN125
- net NEW_158 renamed CLEAN126
- net NEW_159 renamed CLEAN127
- net NEW_16 renamed CLEAN59
- net NEW_161 renamed CLEAN149
- net NEW_167 renamed CLEAN400
- net NEW_168 renamed CLEAN401
- net NEW_169 renamed CLEAN402
- net NEW_170 renamed CLEAN403
- net NEW_173 renamed CLEAN407
- net NEW_177 renamed CLEAN412
- net NEW_178 renamed CLEAN413
- net NEW_179 renamed CLEAN414
- net NEW_186 renamed CLEAN1
- net NEW_187 renamed CLEAN2
- net NEW_188 renamed CLEAN3
- net NEW_19 renamed CLEAN29
- net NEW_191 renamed CLEAN15
- net NEW_193 renamed CLEAN16
- net NEW_200 renamed CLEAN315
- net NEW_201 renamed CLEAN316
- net NEW_202 renamed CLEAN317
- net NEW_203 renamed CLEAN318
- net NEW_204 renamed CLEAN319
- net NEW_21 renamed CLEAN73
- net NEW_210 renamed CLEAN68
- net NEW_214 renamed CLEAN136
- net NEW_215 renamed CLEAN69
- net NEW_216 renamed CLEAN70
- net NEW_22 renamed CLEAN71
- net NEW_222 renamed CLEAN79
- net NEW_223 renamed CLEAN80
- net NEW_224 renamed CLEAN81
- net NEW_226 renamed CLEAN336
- net NEW_227 renamed CLEAN337
- net NEW_228 renamed CLEAN338
- net NEW_229 renamed CLEAN339
- net NEW_23 renamed CLEAN72
- net NEW_233 renamed CLEAN333
- net NEW_238 renamed CLEAN328
- net NEW_239 renamed CLEAN329
- net NEW_240 renamed CLEAN60
- net NEW_246 renamed CLEAN45
- net NEW_248 renamed CLEAN46
- net NEW_250 renamed CLEAN47
- net NEW_251 renamed CLEAN30
- net NEW_252 renamed CLEAN31
- net NEW_255 renamed CLEAN61
- net NEW_256 renamed CLEAN62
- net NEW_257 renamed CLEAN64
- net NEW_258 renamed CLEAN65
- net NEW_259 renamed CLEAN63
- net NEW_26 renamed CLEAN426
- net NEW_261 renamed CLEAN32
- net NEW_265 renamed CLEAN34
- net NEW_266 renamed CLEAN33
- net NEW_268 renamed CLEAN270
- net NEW_27 renamed CLEAN427
- net NEW_270 renamed CLEAN82
- net NEW_271 renamed CLEAN83
- net NEW_274 renamed CLEAN154
- net NEW_28 renamed CLEAN428
- net NEW_282 renamed CLEAN92
- net NEW_283 renamed CLEAN93
- net NEW_284 renamed CLEAN94
- net NEW_29 renamed CLEAN429
- net NEW_290 renamed CLEAN360
- net NEW_292 renamed CLEAN362
- net NEW_293 renamed CLEAN363
- net NEW_294 renamed CLEAN364
- net NEW_298 renamed CLEAN358
- net NEW_299 renamed CLEAN359
- net NEW_30 renamed CLEAN420
- net NEW_301 renamed CLEAN287
- net NEW_304 renamed CLEAN285
- net NEW_306 renamed CLEAN289
- net NEW_309 renamed CLEAN288
- net NEW_311 renamed CLEAN292
- net NEW_319 renamed CLEAN384
- net NEW_321 renamed CLEAN376
- net NEW_323 renamed CLEAN378
- net NEW_325 renamed CLEAN370
- net NEW_327 renamed CLEAN372
- net NEW_328 renamed CLEAN373
- net NEW_330 renamed CLEAN95
- net NEW_331 renamed CLEAN389
- net NEW_333 renamed CLEAN91
- net NEW_337 renamed CLEAN96
- net NEW_341 renamed CLEAN105
- net NEW_342 renamed CLEAN106
- net NEW_343 renamed CLEAN107
- net NEW_344 renamed CLEAN108
- net NEW_347 renamed CLEAN386
- net NEW_35 renamed CLEAN415
- net NEW_352 renamed CLEAN392
- net NEW_353 renamed CLEAN393
- net NEW_354 renamed CLEAN394
- net NEW_355 renamed CLEAN395
- net NEW_356 renamed CLEAN396
- net NEW_357 renamed CLEAN397
- net NEW_358 renamed CLEAN398
- net NEW_36 renamed CLEAN416
- net NEW_361 renamed CLEAN306
- net NEW_362 renamed CLEAN307
- net NEW_363 renamed CLEAN308
- net NEW_364 renamed CLEAN309
- net NEW_365 renamed CLEAN485
- net NEW_367 renamed CLEAN487
- net NEW_369 renamed CLEAN489
- net NEW_37 renamed CLEAN417
- net NEW_370 renamed CLEAN286
- net NEW_372 renamed CLEAN258
- net NEW_374 renamed CLEAN245
- net NEW_376 renamed CLEAN275
- net NEW_377 renamed CLEAN274
- net NEW_379 renamed CLEAN261
- net NEW_38 renamed CLEAN418
- net NEW_380 renamed CLEAN291
- net NEW_381 renamed CLEAN290
- net NEW_382 renamed CLEAN276
- net NEW_384 renamed CLEAN263
- net NEW_385 renamed CLEAN120
- net NEW_386 renamed CLEAN121
- net NEW_387 renamed CLEAN122
- net NEW_390 renamed CLEAN284
- net NEW_391 renamed CLEAN152
- net NEW_393 renamed CLEAN135
- net NEW_397 renamed CLEAN297
- net NEW_398 renamed CLEAN150
- net NEW_399 renamed CLEAN151
- net NEW_40 renamed CLEAN74
- net NEW_402 renamed CLEAN262
- net NEW_405 renamed CLEAN279
- net NEW_408 renamed CLEAN277
- net NEW_409 renamed CLEAN250
- net NEW_410 renamed CLEAN153
- net NEW_413 renamed CLEAN165
- net NEW_414 renamed CLEAN166
- net NEW_416 renamed CLEAN516
- net NEW_418 renamed CLEAN518
- net NEW_420 renamed CLEAN510
- net NEW_422 renamed CLEAN512
- net NEW_423 renamed CLEAN513
- net NEW_426 renamed CLEAN506
- net NEW_429 renamed CLEAN509
- net NEW_43 renamed CLEAN102
- net NEW_431 renamed CLEAN266
- net NEW_433 renamed CLEAN278
- net NEW_437 renamed CLEAN253
- net NEW_438 renamed CLEAN254
- net NEW_44 renamed CLEAN103
- net NEW_441 renamed CLEAN268
- net NEW_442 renamed CLEAN298
- net NEW_443 renamed CLEAN267
- net NEW_444 renamed CLEAN299
- net NEW_447 renamed CLEAN532
- net NEW_450 renamed CLEAN525
- net NEW_452 renamed CLEAN527
- net NEW_453 renamed CLEAN528
- net NEW_454 renamed CLEAN529
- net NEW_455 renamed CLEAN520
- net NEW_457 renamed CLEAN522
- net NEW_459 renamed CLEAN524
- net NEW_466 renamed CLEAN281
- net NEW_469 renamed CLEAN280
- net NEW_472 renamed CLEAN229
- net NEW_473 renamed CLEAN296
- net NEW_476 renamed CLEAN546
- net NEW_477 renamed CLEAN547
- net NEW_48 renamed CLEAN84
- net NEW_480 renamed CLEAN595
- net NEW_481 renamed CLEAN596
- net NEW_482 renamed CLEAN597
- net NEW_485 renamed CLEAN540
- net NEW_487 renamed CLEAN542
- net NEW_489 renamed CLEAN544
- net NEW_49 renamed CLEAN85
- net NEW_490 renamed CLEAN535
- net NEW_495 renamed CLEAN295
- net NEW_499 renamed CLEAN218
- net NEW_50 renamed CLEAN26
- net NEW_500 renamed CLEAN181
- net NEW_501 renamed CLEAN193
- net NEW_502 renamed CLEAN194
- net NEW_504 renamed CLEAN216
- net NEW_505 renamed CLEAN190
- net NEW_506 renamed CLEAN189
- net NEW_508 renamed CLEAN188
- net NEW_513 renamed CLEAN563
- net NEW_514 renamed CLEAN564
- net NEW_518 renamed CLEAN558
- net NEW_520 renamed CLEAN550
- net NEW_524 renamed CLEAN554
- net NEW_525 renamed CLEAN192
- net NEW_529 renamed CLEAN191
- net NEW_53 renamed CLEAN7
- net NEW_530 renamed CLEAN196
- net NEW_54 renamed CLEAN8
- net NEW_541 renamed CLEAN576
- net NEW_543 renamed CLEAN578
- net NEW_544 renamed CLEAN579
- net NEW_545 renamed CLEAN570
- net NEW_547 renamed CLEAN572
- net NEW_548 renamed CLEAN573
- net NEW_549 renamed CLEAN574
- net NEW_55 renamed CLEAN440
- net NEW_553 renamed CLEAN568
- net NEW_554 renamed CLEAN569
- net NEW_555 renamed CLEAN199
- net NEW_556 renamed CLEAN200
- net NEW_557 renamed CLEAN201
- net NEW_558 renamed CLEAN202
- net NEW_559 renamed CLEAN203
- net NEW_56 renamed CLEAN441
- net NEW_560 renamed CLEAN265
- net NEW_561 renamed CLEAN251
- net NEW_563 renamed CLEAN217
- net NEW_564 renamed CLEAN215
- net NEW_565 renamed CLEAN209
- net NEW_569 renamed CLEAN238
- net NEW_57 renamed CLEAN442
- net NEW_570 renamed CLEAN590
- net NEW_571 renamed CLEAN591
- net NEW_572 renamed CLEAN592
- net NEW_574 renamed CLEAN594
- net NEW_577 renamed CLEAN587
- net NEW_58 renamed CLEAN443
- net NEW_580 renamed CLEAN580
- net NEW_581 renamed CLEAN581
- net NEW_583 renamed CLEAN583
- net NEW_586 renamed CLEAN234
- net NEW_587 renamed CLEAN233
- net NEW_589 renamed CLEAN225
- net NEW_591 renamed CLEAN221
- net NEW_593 renamed CLEAN211
- net NEW_596 renamed CLEAN220
- net NEW_597 renamed CLEAN212
- net NEW_599 renamed CLEAN0
- net NEW_64 renamed CLEAN439
- net NEW_65 renamed CLEAN430
- net NEW_66 renamed CLEAN431
- net NEW_67 renamed CLEAN432
- net NEW_68 renamed CLEAN433
- net NEW_69 renamed CLEAN434
- net NEW_70 renamed CLEAN86
- net NEW_71 renamed CLEAN87
- net NEW_73 renamed CLEAN41
- net NEW_74 renamed CLEAN42
- net NEW_75 renamed CLEAN88
- net NEW_8 renamed CLEAN404
- net NEW_80 renamed CLEAN128
- net NEW_81 renamed CLEAN129
- net NEW_82 renamed CLEAN130
- net NEW_83 renamed CLEAN99
- net NEW_84 renamed CLEAN100
- net NEW_85 renamed CLEAN455
- net NEW_86 renamed CLEAN456
- net NEW_87 renamed CLEAN457
- net NEW_92 renamed CLEAN452
- net NEW_95 renamed CLEAN445
- net NEW_96 renamed CLEAN446
- net NEW_97 renamed CLEAN447
- net NEW_98 renamed CLEAN448
- removed net NEW_0: JP1.10, JP42.1
- removed net NEW_1: JP1.11, JP42.2
- removed net NEW_118: JP109.4, JP15.8
- removed net NEW_119: JP109.5, JP15.6
- removed net NEW_122: JP108.3, JP19.7
- removed net NEW_123: JP108.4, JP19.8
- removed net NEW_124: JP108.5, JP19.9
- removed net NEW_125: JP107.1, JP19.10
- removed net NEW_126: JP107.2, JP19.11
- removed net NEW_127: JP107.3, JP19.12
- removed net NEW_128: JP107.4, JP19.13
- removed net NEW_129: JP107.5, JP19.14
- removed net NEW_145: JP114.1, JP5.10
- removed net NEW_150: JP113.1, JP9.7
- removed net NEW_151: JP113.2, JP9.8
- removed net NEW_171: JP21.12, JP84.1
- removed net NEW_172: JP21.10, JP84.2
- removed net NEW_174: JP21.11, JP84.4
- removed net NEW_175: JP21.14, JP84.5
- removed net NEW_176: JP21.13, JP85.1
- removed net NEW_195: JP49.1, JP7.4
- removed net NEW_196: JP49.2, JP7.7
- removed net NEW_197: JP49.3, JP7.6
- removed net NEW_198: JP49.4, JP7.5
- removed net NEW_199: JP49.5, JP7.8
- removed net NEW_2: JP1.6, JP42.3
- removed net NEW_205: JP3.3, JP47.1
- removed net NEW_206: JP3.5, JP47.2
- removed net NEW_207: JP3.4, JP47.3
- removed net NEW_208: JP3.6, JP47.4
- removed net NEW_209: JP3.7, JP47.5
- removed net NEW_225: JP21.15, JP55.1
- removed net NEW_230: JP19.3, JP54.1
- removed net NEW_231: JP23.8, JP54.2
- removed net NEW_232: JP23.9, JP54.3
- removed net NEW_234: JP23.10, JP54.5
- removed net NEW_235: JP19.4, JP53.1
- removed net NEW_236: JP19.5, JP53.2
- removed net NEW_237: JP19.6, JP53.3
- removed net NEW_25: JP1.14, JP91.1
- removed net NEW_285: JP23.12, JP67.1
- removed net NEW_286: JP23.13, JP67.2
- removed net NEW_287: JP23.11, JP67.3
- removed net NEW_288: JP23.14, JP67.4
- removed net NEW_289: JP23.15, JP67.5
- removed net NEW_291: JP21.7, JP66.2
- removed net NEW_295: JP21.6, JP65.1
- removed net NEW_296: JP21.9, JP65.2
- removed net NEW_297: JP21.8, JP65.3
- removed net NEW_3: JP1.5, JP42.4
- removed net NEW_31: JP3.8, JP90.2
- removed net NEW_315: JP11.1, JP73.1
- removed net NEW_316: JP11.2, JP73.2
- removed net NEW_317: JP11.3, JP73.3
- removed net NEW_318: JP11.4, JP73.4
- removed net NEW_32: JP3.10, JP90.3
- removed net NEW_320: JP35.2, JP72.1
- removed net NEW_322: JP35.1, JP72.3
- removed net NEW_324: JP13.1, JP72.5
- removed net NEW_326: JP37.2, JP71.2
- removed net NEW_329: JP35.3, JP71.5
- removed net NEW_33: JP3.11, JP90.4
- removed net NEW_34: JP3.9, JP90.5
- removed net NEW_346: JP23.3, JP77.1
- removed net NEW_348: JP23.4, JP77.3
- removed net NEW_349: JP23.5, JP77.4
- removed net NEW_350: JP23.6, JP78.1
- removed net NEW_351: JP23.7, JP78.2
- removed net NEW_359: JP25.6, JP79.5
- removed net NEW_360: JP15.5, JP43.1
- removed net NEW_366: JP115.2, JP33.5
- removed net NEW_368: JP115.4, JP33.4
- removed net NEW_39: JP5.11, JP89.5
- removed net NEW_4: JP1.7, JP42.5
- removed net NEW_415: JP127.1, JP33.3
- removed net NEW_417: JP127.3, JP37.14
- removed net NEW_419: JP127.5, JP35.15
- removed net NEW_421: JP126.2, JP33.1
- removed net NEW_424: JP126.5, JP33.2
- removed net NEW_425: JP125.1, JP33.9
- removed net NEW_427: JP125.3, JP37.4
- removed net NEW_428: JP125.4, JP37.3
- removed net NEW_445: JP133.1, JP31.8
- removed net NEW_446: JP133.2, JP31.2
- removed net NEW_448: JP133.4, JP31.7
- removed net NEW_449: JP133.5, JP31.3
- removed net NEW_451: JP132.2, JP31.11
- removed net NEW_456: JP131.2, JP31.13
- removed net NEW_458: JP131.4, JP33.10
- removed net NEW_475: JP139.1, JP37.13
- removed net NEW_478: JP139.4, JP39.9
- removed net NEW_479: JP139.5, JP39.10
- removed net NEW_483: JP161.4, JP31.6
- removed net NEW_484: JP161.5, JP31.4
- removed net NEW_486: JP138.2, JP25.3
- removed net NEW_488: JP138.4, JP25.1
- removed net NEW_491: JP137.2, JP25.5
- removed net NEW_492: JP137.3, JP25.4
- removed net NEW_493: JP137.4, JP25.7
- removed net NEW_494: JP137.5, JP25.8
- removed net NEW_510: JP145.1, JP29.15
- removed net NEW_511: JP145.2, JP27.1
- removed net NEW_512: JP145.3, JP35.10
- removed net NEW_515: JP144.1, JP29.13
- removed net NEW_516: JP144.2, JP29.1
- removed net NEW_517: JP144.3, JP31.12
- removed net NEW_519: JP144.5, JP29.14
- removed net NEW_521: JP143.2, JP29.10
- removed net NEW_522: JP143.3, JP35.5
- removed net NEW_523: JP143.4, JP35.6
- removed net NEW_540: JP151.1, JP29.4
- removed net NEW_542: JP151.3, JP33.8
- removed net NEW_546: JP150.2, JP29.5
- removed net NEW_550: JP149.1, JP27.3
- removed net NEW_551: JP149.2, JP27.4
- removed net NEW_552: JP149.3, JP27.14
- removed net NEW_573: JP157.4, JP27.10
- removed net NEW_575: JP156.1, JP27.11
- removed net NEW_576: JP156.2, JP27.12
- removed net NEW_578: JP156.4, JP31.15
- removed net NEW_579: JP156.5, JP27.13
- removed net NEW_582: JP155.3, JP33.13
- removed net NEW_584: JP155.5, JP33.7
- removed net NEW_59: JP15.11, JP97.5
- removed net NEW_6: JP11.15, JP85.2
- removed net NEW_60: JP15.13, JP96.1
- removed net NEW_61: JP15.14, JP96.2
- removed net NEW_62: JP15.12, JP96.3
- removed net NEW_63: JP15.15, JP96.4
- removed net NEW_7: JP1.12, JP113.4
- removed net NEW_88: JP103.4, JP5.6
- removed net NEW_89: JP103.5, JP5.7
- removed net NEW_9: JP1.13, JP113.5
- removed net NEW_90: JP102.1, JP5.15
- removed net NEW_91: JP102.2, JP5.14
- removed net NEW_93: JP102.4, JP5.8
- removed net NEW_94: JP102.5, JP5.9
- removed net NEW_99: JP101.5, JP7.9
- new net CLEAN10: JP1.11
- new net CLEAN109: JP15.5
- new net CLEAN11: JP1.12
- new net CLEAN110: JP15.6
- new net CLEAN112: JP15.8
- new net CLEAN115: JP15.11
- new net CLEAN116: JP15.12
- new net CLEAN117: JP15.13
- new net CLEAN118: JP15.14
- new net CLEAN119: JP15.15
- new net CLEAN12: JP1.13
- new net CLEAN13: JP1.14
- new net CLEAN137: JP19.3
- new net CLEAN138: JP19.4
- new net CLEAN139: JP19.5
- new net CLEAN140: JP19.6
- new net CLEAN141: JP19.7
- new net CLEAN142: JP19.8
- new net CLEAN143: JP19.9
- new net CLEAN144: JP19.10
- new net CLEAN145: JP19.11
- new net CLEAN146: JP19.12
- new net CLEAN147: JP19.13
- new net CLEAN148: JP19.14
- new net CLEAN155: JP21.6
- new net CLEAN156: JP21.7
- new net CLEAN157: JP21.8
- new net CLEAN158: JP21.9
- new net CLEAN159: JP21.10
- new net CLEAN160: JP21.11
- new net CLEAN161: JP21.12
- new net CLEAN162: JP21.13
- new net CLEAN163: JP21.14
- new net CLEAN164: JP21.15
- new net CLEAN167: JP23.3
- new net CLEAN168: JP23.4
- new net CLEAN169: JP23.5
- new net CLEAN17: JP3.3
- new net CLEAN170: JP23.6
- new net CLEAN171: JP23.7
- new net CLEAN172: JP23.8
- new net CLEAN173: JP23.9
- new net CLEAN174: JP23.10
- new net CLEAN175: JP23.11
- new net CLEAN176: JP23.12
- new net CLEAN177: JP23.13
- new net CLEAN178: JP23.14
- new net CLEAN179: JP23.15
- new net CLEAN18: JP3.4
- new net CLEAN180: JP25.1
- new net CLEAN182: JP25.3
- new net CLEAN183: JP25.4
- new net CLEAN184: JP25.5
- new net CLEAN185: JP25.6
- new net CLEAN186: JP25.7
- new net CLEAN187: JP25.8
- new net CLEAN19: JP3.5
- new net CLEAN195: JP27.1
- new net CLEAN197: JP27.3
- new net CLEAN198: JP27.4
- new net CLEAN20: JP3.6
- new net CLEAN204: JP27.10
- new net CLEAN205: JP27.11
- new net CLEAN206: JP27.12
- new net CLEAN207: JP27.13
- new net CLEAN208: JP27.14
- new net CLEAN21: JP3.7
- new net CLEAN210: JP29.1
- new net CLEAN213: JP29.4
- new net CLEAN214: JP29.5
- new net CLEAN219: JP29.10
- new net CLEAN22: JP3.8
- new net CLEAN222: JP29.13
- new net CLEAN223: JP29.14
- new net CLEAN224: JP29.15
- new net CLEAN226: JP31.2
- new net CLEAN227: JP31.3
- new net CLEAN228: JP31.4
- new net CLEAN23: JP3.9
- new net CLEAN230: JP31.6
- new net CLEAN231: JP31.7
- new net CLEAN232: JP31.8
- new net CLEAN235: JP31.11
- new net CLEAN236: JP31.12
- new net CLEAN237: JP31.13
- new net CLEAN239: JP31.15
- new net CLEAN24: JP3.10
- new net CLEAN240: JP33.1
- new net CLEAN241: JP33.2
- new net CLEAN242: JP33.3
- new net CLEAN243: JP33.4
- new net CLEAN244: JP33.5
- new net CLEAN246: JP33.7
- new net CLEAN247: JP33.8
- new net CLEAN248: JP33.9
- new net CLEAN249: JP33.10
- new net CLEAN25: JP3.11
- new net CLEAN252: JP33.13
- new net CLEAN255: JP35.1
- new net CLEAN256: JP35.2
- new net CLEAN257: JP35.3
- new net CLEAN259: JP35.5
- new net CLEAN260: JP35.6
- new net CLEAN264: JP35.10
- new net CLEAN269: JP35.15
- new net CLEAN271: JP37.2
- new net CLEAN272: JP37.3
- new net CLEAN273: JP37.4
- new net CLEAN282: JP37.13
- new net CLEAN283: JP37.14
- new net CLEAN293: JP39.9
- new net CLEAN294: JP39.10
- new net CLEAN300: JP42.1
- new net CLEAN301: JP42.2
- new net CLEAN302: JP42.3
- new net CLEAN303: JP42.4
- new net CLEAN304: JP42.5
- new net CLEAN305: JP43.1
- new net CLEAN310: JP47.1
- new net CLEAN311: JP47.2
- new net CLEAN312: JP47.3
- new net CLEAN313: JP47.4
- new net CLEAN314: JP47.5
- new net CLEAN320: JP49.1
- new net CLEAN321: JP49.2
- new net CLEAN322: JP49.3
- new net CLEAN323: JP49.4
- new net CLEAN324: JP49.5
- new net CLEAN325: JP53.1
- new net CLEAN326: JP53.2
- new net CLEAN327: JP53.3
- new net CLEAN330: JP54.1
- new net CLEAN331: JP54.2
- new net CLEAN332: JP54.3
- new net CLEAN334: JP54.5
- new net CLEAN335: JP55.1
- new net CLEAN35: JP5.6
- new net CLEAN355: JP65.1
- new net CLEAN356: JP65.2
- new net CLEAN357: JP65.3
- new net CLEAN36: JP5.7
- new net CLEAN361: JP66.2
- new net CLEAN365: JP67.1
- new net CLEAN366: JP67.2
- new net CLEAN367: JP67.3
- new net CLEAN368: JP67.4
- new net CLEAN369: JP67.5
- new net CLEAN37: JP5.8
- new net CLEAN371: JP71.2
- new net CLEAN374: JP71.5
- new net CLEAN375: JP72.1
- new net CLEAN377: JP72.3
- new net CLEAN379: JP72.5
- new net CLEAN38: JP5.9
- new net CLEAN380: JP73.1
- new net CLEAN381: JP73.2
- new net CLEAN382: JP73.3
- new net CLEAN383: JP73.4
- new net CLEAN385: JP77.1
- new net CLEAN387: JP77.3
- new net CLEAN388: JP77.4
- new net CLEAN39: JP5.10
- new net CLEAN390: JP78.1
- new net CLEAN391: JP78.2
- new net CLEAN399: JP79.5
- new net CLEAN4: JP1.5
- new net CLEAN40: JP5.11
- new net CLEAN405: JP84.1
- new net CLEAN406: JP84.2
- new net CLEAN408: JP84.4
- new net CLEAN409: JP84.5
- new net CLEAN410: JP85.1
- new net CLEAN411: JP85.2
- new net CLEAN419: JP89.5
- new net CLEAN421: JP90.2
- new net CLEAN422: JP90.3
- new net CLEAN423: JP90.4
- new net CLEAN424: JP90.5
- new net CLEAN425: JP91.1
- new net CLEAN43: JP5.14
- new net CLEAN435: JP96.1
- new net CLEAN436: JP96.2
- new net CLEAN437: JP96.3
- new net CLEAN438: JP96.4
- new net CLEAN44: JP5.15
- new net CLEAN444: JP97.5
- new net CLEAN449: JP101.5
- new net CLEAN450: JP102.1
- new net CLEAN451: JP102.2
- new net CLEAN453: JP102.4
- new net CLEAN454: JP102.5
- new net CLEAN458: JP103.4
- new net CLEAN459: JP103.5
- new net CLEAN460: JP107.1
- new net CLEAN461: JP107.2
- new net CLEAN462: JP107.3
- new net CLEAN463: JP107.4
- new net CLEAN464: JP107.5
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
Commit message: Routed Files
Connections:
- net CLEAN305 renamed 0_1438933749
- net CLEAN380 renamed 0_1438936495
- removed net CLEAN0: JP1.1
- removed net CLEAN1: JP1.2
- removed net CLEAN10: JP1.11
- removed net CLEAN100: JP13.11
- removed net CLEAN101: JP13.12
- removed net CLEAN102: JP13.13
- removed net CLEAN103: JP13.14
- removed net CLEAN105: JP15.1
- removed net CLEAN106: JP15.2
- removed net CLEAN107: JP15.3
- removed net CLEAN108: JP15.4
- removed net CLEAN109: JP15.5
- removed net CLEAN11: JP1.12
- removed net CLEAN110: JP15.6
- removed net CLEAN111: JP15.7
- removed net CLEAN112: JP15.8
- removed net CLEAN113: JP15.9
- removed net CLEAN114: JP15.10
- removed net CLEAN115: JP15.11
- removed net CLEAN116: JP15.12
- removed net CLEAN117: JP15.13
- removed net CLEAN118: JP15.14
- removed net CLEAN119: JP15.15
- removed net CLEAN12: JP1.13
- removed net CLEAN120: JP17.1
- removed net CLEAN121: JP17.2
- removed net CLEAN122: JP17.3
- removed net CLEAN123: JP17.4
- removed net CLEAN124: JP17.5
- removed net CLEAN125: JP17.6
- removed net CLEAN126: JP17.7
- removed net CLEAN127: JP17.8
- removed net CLEAN128: JP17.9
- removed net CLEAN129: JP17.10
- removed net CLEAN13: JP1.14
- removed net CLEAN130: JP17.11
- removed net CLEAN131: JP17.12
- removed net CLEAN132: JP17.13
- removed net CLEAN133: JP17.14
- removed net CLEAN134: JP17.15
- removed net CLEAN135: JP19.1
- removed net CLEAN136: JP19.2
- removed net CLEAN137: JP19.3
- removed net CLEAN138: JP19.4
- removed net CLEAN139: JP19.5
- removed net CLEAN14: JP1.15
- removed net CLEAN140: JP19.6
- removed net CLEAN141: JP19.7
- removed net CLEAN142: JP19.8
- removed net CLEAN143: JP19.9
- removed net CLEAN144: JP19.10
- removed net CLEAN145: JP19.11
- removed net CLEAN146: JP19.12
- removed net CLEAN147: JP19.13
- removed net CLEAN148: JP19.14
- removed net CLEAN149: JP19.15
- removed net CLEAN15: JP3.1
- removed net CLEAN150: JP21.1
- removed net CLEAN151: JP21.2
- removed net CLEAN152: JP21.3
- removed net CLEAN153: JP21.4
- removed net CLEAN154: JP21.5
- removed net CLEAN155: JP21.6
- removed net CLEAN156: JP21.7
- removed net CLEAN157: JP21.8
- removed net CLEAN158: JP21.9
- removed net CLEAN159: JP21.10
- removed net CLEAN16: JP3.2
- removed net CLEAN160: JP21.11
- removed net CLEAN161: JP21.12
- removed net CLEAN162: JP21.13
- removed net CLEAN163: JP21.14
- removed net CLEAN164: JP21.15
- removed net CLEAN165: JP23.1
- removed net CLEAN166: JP23.2
- removed net CLEAN167: JP23.3
- removed net CLEAN168: JP23.4
- removed net CLEAN169: JP23.5
- removed net CLEAN17: JP3.3
- removed net CLEAN170: JP23.6
- removed net CLEAN171: JP23.7
- removed net CLEAN172: JP23.8
- removed net CLEAN173: JP23.9
- removed net CLEAN174: JP23.10
- removed net CLEAN175: JP23.11
- removed net CLEAN176: JP23.12
- removed net CLEAN177: JP23.13
- removed net CLEAN178: JP23.14
- removed net CLEAN179: JP23.15
- removed net CLEAN18: JP3.4
- removed net CLEAN180: JP25.1
- removed net CLEAN181: JP25.2
- removed net CLEAN182: JP25.3
- removed net CLEAN183: JP25.4
- removed net CLEAN184: JP25.5
- removed net CLEAN185: JP25.6
- removed net CLEAN186: JP25.7
- removed net CLEAN187: JP25.8
- removed net CLEAN188: JP25.9
- removed net CLEAN189: JP25.10
- removed net CLEAN19: JP3.5
- removed net CLEAN190: JP25.11
- removed net CLEAN191: JP25.12
- removed net CLEAN192: JP25.13
- removed net CLEAN193: JP25.14
- removed net CLEAN194: JP25.15
- removed net CLEAN195: JP27.1
- removed net CLEAN196: JP27.2
- removed net CLEAN197: JP27.3
- removed net CLEAN198: JP27.4
- removed net CLEAN199: JP27.5
- removed net CLEAN2: JP1.3
- removed net CLEAN20: JP3.6
- removed net CLEAN200: JP27.6
- removed net CLEAN201: JP27.7
- removed net CLEAN202: JP27.8
- removed net CLEAN203: JP27.9
- removed net CLEAN204: JP27.10
- removed net CLEAN205: JP27.11
- removed net CLEAN206: JP27.12
- removed net CLEAN207: JP27.13
- removed net CLEAN208: JP27.14
- removed net CLEAN209: JP27.15
- removed net CLEAN21: JP3.7
- removed net CLEAN210: JP29.1
- removed net CLEAN211: JP29.2
- removed net CLEAN212: JP29.3
- removed net CLEAN213: JP29.4
- removed net CLEAN214: JP29.5
- removed net CLEAN215: JP29.6
- removed net CLEAN216: JP29.7
- removed net CLEAN217: JP29.8
- removed net CLEAN218: JP29.9
- removed net CLEAN219: JP29.10
- removed net CLEAN22: JP3.8
- removed net CLEAN220: JP29.11
- removed net CLEAN221: JP29.12
- removed net CLEAN222: JP29.13
- removed net CLEAN223: JP29.14
- removed net CLEAN224: JP29.15
- removed net CLEAN225: JP31.1
- removed net CLEAN226: JP31.2
- removed net CLEAN227: JP31.3
- removed net CLEAN228: JP31.4
- removed net CLEAN229: JP31.5
- removed net CLEAN23: JP3.9
- removed net CLEAN230: JP31.6
- removed net CLEAN231: JP31.7
- removed net CLEAN232: JP31.8
- removed net CLEAN233: JP31.9
- removed net CLEAN234: JP31.10
- removed net CLEAN235: JP31.11
- removed net CLEAN236: JP31.12
- removed net CLEAN237: JP31.13
- removed net CLEAN238: JP31.14
- removed net CLEAN239: JP31.15
- removed net CLEAN24: JP3.10
- removed net CLEAN240: JP33.1
- removed net CLEAN241: JP33.2
- removed net CLEAN242: JP33.3
- removed net CLEAN243: JP33.4
- removed net CLEAN244: JP33.5
- removed net CLEAN245: JP33.6
- removed net CLEAN246: JP33.7
- removed net CLEAN247: JP33.8
- removed net CLEAN248: JP33.9
- removed net CLEAN249: JP33.10
- removed net CLEAN250: JP33.11
- removed net CLEAN251: JP33.12
- removed net CLEAN252: JP33.13
- removed net CLEAN253: JP33.14
- removed net CLEAN254: JP33.15
- removed net CLEAN256: JP35.2
- removed net CLEAN257: JP35.3
- removed net CLEAN258: JP35.4
- removed net CLEAN259: JP35.5
- removed net CLEAN26: JP3.12
- removed net CLEAN260: JP35.6
- removed net CLEAN261: JP35.7
- removed net CLEAN262: JP35.8
- removed net CLEAN263: JP35.9
- removed net CLEAN264: JP35.10
- removed net CLEAN265: JP35.11
- removed net CLEAN266: JP35.12
- removed net CLEAN267: JP35.13
- removed net CLEAN268: JP35.14
- removed net CLEAN269: JP35.15
- removed net CLEAN27: JP3.13
- removed net CLEAN270: JP37.1
- removed net CLEAN271: JP37.2
- removed net CLEAN272: JP37.3
- removed net CLEAN273: JP37.4
- removed net CLEAN274: JP37.5
- removed net CLEAN275: JP37.6
- removed net CLEAN276: JP37.7
- removed net CLEAN277: JP37.8
- removed net CLEAN278: JP37.9
- removed net CLEAN279: JP37.10
- removed net CLEAN28: JP3.14
- removed net CLEAN280: JP37.11
- removed net CLEAN281: JP37.12
- removed net CLEAN282: JP37.13
- removed net CLEAN283: JP37.14
- removed net CLEAN284: JP37.15
- removed net CLEAN285: JP39.1
- removed net CLEAN286: JP39.2
- removed net CLEAN287: JP39.3
- removed net CLEAN288: JP39.4
- removed net CLEAN289: JP39.5
- removed net CLEAN29: JP3.15
- removed net CLEAN290: JP39.6
- removed net CLEAN291: JP39.7
- removed net CLEAN292: JP39.8
- removed net CLEAN293: JP39.9
- removed net CLEAN294: JP39.10
- removed net CLEAN295: JP39.11
- removed net CLEAN296: JP39.12
- removed net CLEAN297: JP39.13
- removed net CLEAN298: JP39.14
- removed net CLEAN299: JP39.15
- removed net CLEAN3: JP1.4
- removed net CLEAN30: JP5.1
- removed net CLEAN300: JP42.1
- removed net CLEAN301: JP42.2
- removed net CLEAN302: JP42.3
- removed net CLEAN303: JP42.4
- removed net CLEAN304: JP42.5
- removed net CLEAN306: JP43.2
- removed net CLEAN307: JP43.3
- removed net CLEAN308: JP43.4
- removed net CLEAN309: JP43.5
- removed net CLEAN31: JP5.2
- removed net CLEAN310: JP47.1
- removed net CLEAN311: JP47.2
- removed net CLEAN312: JP47.3
- removed net CLEAN313: JP47.4
- removed net CLEAN314: JP47.5
- removed net CLEAN315: JP48.1
- removed net CLEAN316: JP48.2
- removed net CLEAN317: JP48.3
- removed net CLEAN318: JP48.4
- removed net CLEAN319: JP48.5
- removed net CLEAN32: JP5.3
- removed net CLEAN320: JP49.1
- removed net CLEAN321: JP49.2
- removed net CLEAN322: JP49.3
- removed net CLEAN323: JP49.4
- removed net CLEAN324: JP49.5
- removed net CLEAN325: JP53.1
- removed net CLEAN326: JP53.2
- removed net CLEAN327: JP53.3
- removed net CLEAN328: JP53.4
- removed net CLEAN329: JP53.5
- removed net CLEAN33: JP5.4
- removed net CLEAN330: JP54.1
- removed net CLEAN331: JP54.2
- removed net CLEAN332: JP54.3
- removed net CLEAN333: JP54.4
- removed net CLEAN334: JP54.5
- removed net CLEAN335: JP55.1
- removed net CLEAN336: JP55.2
- removed net CLEAN337: JP55.3
- removed net CLEAN338: JP55.4
- removed net CLEAN339: JP55.5
- removed net CLEAN34: JP5.5
- removed net CLEAN340: JP59.1
- removed net CLEAN341: JP59.2
- removed net CLEAN342: JP59.3
- removed net CLEAN343: JP59.4
- removed net CLEAN344: JP59.5
- removed net CLEAN345: JP60.1
- removed net CLEAN346: JP60.2
- removed net CLEAN347: JP60.3
- removed net CLEAN348: JP60.4
- removed net CLEAN349: JP60.5
- removed net CLEAN35: JP5.6
- removed net CLEAN350: JP61.1
- removed net CLEAN351: JP61.2
- removed net CLEAN352: JP61.3
- removed net CLEAN353: JP61.4
- removed net CLEAN354: JP61.5
- removed net CLEAN355: JP65.1
- removed net CLEAN356: JP65.2
- removed net CLEAN357: JP65.3
- removed net CLEAN358: JP65.4
- removed net CLEAN359: JP65.5
- removed net CLEAN36: JP5.7
- removed net CLEAN360: JP66.1
- removed net CLEAN361: JP66.2
- removed net CLEAN362: JP66.3
- removed net CLEAN363: JP66.4
- removed net CLEAN364: JP66.5
- removed net CLEAN365: JP67.1
- removed net CLEAN366: JP67.2
- removed net CLEAN367: JP67.3
- removed net CLEAN368: JP67.4
- removed net CLEAN369: JP67.5
- removed net CLEAN37: JP5.8
- removed net CLEAN370: JP71.1
- removed net CLEAN371: JP71.2
- removed net CLEAN372: JP71.3
- removed net CLEAN373: JP71.4
- removed net CLEAN374: JP71.5
- removed net CLEAN375: JP72.1
- removed net CLEAN376: JP72.2
- removed net CLEAN377: JP72.3
- removed net CLEAN378: JP72.4
- removed net CLEAN379: JP72.5
- removed net CLEAN38: JP5.9
- removed net CLEAN381: JP73.2
- removed net CLEAN382: JP73.3
- removed net CLEAN383: JP73.4
- removed net CLEAN384: JP73.5
- removed net CLEAN385: JP77.1
- removed net CLEAN386: JP77.2
- removed net CLEAN387: JP77.3
- removed net CLEAN388: JP77.4
- removed net CLEAN389: JP77.5
- removed net CLEAN39: JP5.10
- removed net CLEAN390: JP78.1
- removed net CLEAN391: JP78.2
- removed net CLEAN392: JP78.3
- removed net CLEAN393: JP78.4
- removed net CLEAN394: JP78.5
- removed net CLEAN395: JP79.1
- removed net CLEAN396: JP79.2
- removed net CLEAN397: JP79.3
- removed net CLEAN398: JP79.4
- removed net CLEAN399: JP79.5
- removed net CLEAN4: JP1.5
- removed net CLEAN40: JP5.11
- removed net CLEAN400: JP83.1
- removed net CLEAN401: JP83.2
- removed net CLEAN402: JP83.3
- removed net CLEAN403: JP83.4
- removed net CLEAN404: JP83.5
- removed net CLEAN405: JP84.1
- removed net CLEAN406: JP84.2
- removed net CLEAN407: JP84.3
- removed net CLEAN408: JP84.4
- removed net CLEAN409: JP84.5
- removed net CLEAN41: JP5.12
- removed net CLEAN410: JP85.1
- removed net CLEAN411: JP85.2
- removed net CLEAN412: JP85.3
- removed net CLEAN413: JP85.4
- removed net CLEAN414: JP85.5
- removed net CLEAN415: JP89.1
- removed net CLEAN416: JP89.2
- removed net CLEAN417: JP89.3
- removed net CLEAN418: JP89.4
- removed net CLEAN419: JP89.5
- removed net CLEAN42: JP5.13
- removed net CLEAN420: JP90.1
- removed net CLEAN421: JP90.2
- removed net CLEAN422: JP90.3
- removed net CLEAN423: JP90.4
- removed net CLEAN424: JP90.5
- removed net CLEAN425: JP91.1
- removed net CLEAN426: JP91.2
- removed net CLEAN427: JP91.3
- removed net CLEAN428: JP91.4
- removed net CLEAN429: JP91.5
- removed net CLEAN43: JP5.14
- removed net CLEAN430: JP95.1
- removed net CLEAN431: JP95.2
- removed net CLEAN432: JP95.3
- removed net CLEAN433: JP95.4
- removed net CLEAN434: JP95.5
- removed net CLEAN435: JP96.1
- removed net CLEAN436: JP96.2
- removed net CLEAN437: JP96.3
- removed net CLEAN438: JP96.4
- removed net CLEAN439: JP96.5
- removed net CLEAN44: JP5.15
- removed net CLEAN440: JP97.1
- removed net CLEAN441: JP97.2
- removed net CLEAN442: JP97.3
- removed net CLEAN443: JP97.4
- removed net CLEAN444: JP97.5
- removed net CLEAN445: JP101.1
- removed net CLEAN446: JP101.2
- removed net CLEAN447: JP101.3
- removed net CLEAN448: JP101.4
- removed net CLEAN449: JP101.5
- removed net CLEAN45: JP7.1
- removed net CLEAN450: JP102.1
- removed net CLEAN451: JP102.2
- removed net CLEAN452: JP102.3
- removed net CLEAN453: JP102.4
- removed net CLEAN454: JP102.5
- removed net CLEAN455: JP103.1
- removed net CLEAN456: JP103.2
- removed net CLEAN457: JP103.3
- removed net CLEAN458: JP103.4
- removed net CLEAN459: JP103.5
- removed net CLEAN46: JP7.2
- removed net CLEAN460: JP107.1
- removed net CLEAN461: JP107.2
- removed net CLEAN462: JP107.3
- removed net CLEAN463: JP107.4
- removed net CLEAN464: JP107.5
- removed net CLEAN465: JP108.1
- removed net CLEAN466: JP108.2
- removed net CLEAN467: JP108.3
- removed net CLEAN468: JP108.4
- removed net CLEAN469: JP108.5
- removed net CLEAN47: JP7.3
- removed net CLEAN470: JP109.1
- removed net CLEAN471: JP109.2
- removed net CLEAN472: JP109.3
- removed net CLEAN473: JP109.4
- removed net CLEAN474: JP109.5
- removed net CLEAN475: JP113.1
- removed net CLEAN476: JP113.2
- removed net CLEAN477: JP113.3
- removed net CLEAN478: JP113.4
- removed net CLEAN479: JP113.5
- removed net CLEAN48: JP7.4
- removed net CLEAN480: JP114.1
- removed net CLEAN481: JP114.2
- removed net CLEAN482: JP114.3
- removed net CLEAN483: JP114.4
- removed net CLEAN484: JP114.5
- removed net CLEAN485: JP115.1
- removed net CLEAN486: JP115.2
- removed net CLEAN487: JP115.3
- removed net CLEAN488: JP115.4
- removed net CLEAN489: JP115.5
- removed net CLEAN49: JP7.5
- removed net CLEAN490: JP119.1
- removed net CLEAN491: JP119.2
- removed net CLEAN492: JP119.3
- removed net CLEAN493: JP119.4
- removed net CLEAN494: JP119.5
- removed net CLEAN495: JP120.1
- removed net CLEAN496: JP120.2
- removed net CLEAN497: JP120.3
- removed net CLEAN498: JP120.4
- removed net CLEAN499: JP120.5
- removed net CLEAN5: JP1.6
- removed net CLEAN50: JP7.6
- removed net CLEAN500: JP121.1
- removed net CLEAN501: JP121.2
- removed net CLEAN502: JP121.3
- removed net CLEAN503: JP121.4
- removed net CLEAN504: JP121.5
- removed net CLEAN505: JP125.1
- removed net CLEAN506: JP125.2
- removed net CLEAN507: JP125.3
- removed net CLEAN508: JP125.4
- removed net CLEAN509: JP125.5
- removed net CLEAN51: JP7.7
- removed net CLEAN510: JP126.1
- removed net CLEAN511: JP126.2
- removed net CLEAN512: JP126.3
- removed net CLEAN513: JP126.4
- removed net CLEAN514: JP126.5
- removed net CLEAN515: JP127.1
- removed net CLEAN516: JP127.2
- removed net CLEAN517: JP127.3
- removed net CLEAN518: JP127.4
- removed net CLEAN52: JP7.8
- removed net CLEAN520: JP131.1
- removed net CLEAN521: JP131.2
- removed net CLEAN522: JP131.3
- removed net CLEAN523: JP131.4
- removed net CLEAN524: JP131.5
- removed net CLEAN525: JP132.1
- removed net CLEAN526: JP132.2
- removed net CLEAN527: JP132.3
- removed net CLEAN528: JP132.4
- removed net CLEAN529: JP132.5
- removed net CLEAN53: JP7.9
- removed net CLEAN530: JP133.1
- removed net CLEAN531: JP133.2
- removed net CLEAN532: JP133.3
- removed net CLEAN533: JP133.4
- removed net CLEAN534: JP133.5
- removed net CLEAN535: JP137.1
- removed net CLEAN536: JP137.2
- removed net CLEAN537: JP137.3
- removed net CLEAN538: JP137.4
- removed net CLEAN539: JP137.5
- removed net CLEAN54: JP7.10
- removed net CLEAN540: JP138.1
- removed net CLEAN541: JP138.2
- removed net CLEAN542: JP138.3
- removed net CLEAN543: JP138.4
- removed net CLEAN544: JP138.5
- removed net CLEAN545: JP139.1
- removed net CLEAN546: JP139.2
- removed net CLEAN547: JP139.3
- removed net CLEAN548: JP139.4
- removed net CLEAN549: JP139.5
- removed net CLEAN55: JP7.11
- removed net CLEAN550: JP143.1
- removed net CLEAN551: JP143.2
- removed net CLEAN552: JP143.3
- removed net CLEAN553: JP143.4
- removed net CLEAN554: JP143.5
- removed net CLEAN555: JP144.1
- removed net CLEAN556: JP144.2
- removed net CLEAN557: JP144.3
- removed net CLEAN558: JP144.4
- removed net CLEAN559: JP144.5
- removed net CLEAN56: JP7.12
- removed net CLEAN560: JP145.1
- removed net CLEAN561: JP145.2
- removed net CLEAN562: JP145.3
- removed net CLEAN563: JP145.4
- removed net CLEAN564: JP145.5
- removed net CLEAN565: JP149.1
- removed net CLEAN566: JP149.2
- removed net CLEAN567: JP149.3
- removed net CLEAN568: JP149.4
- removed net CLEAN569: JP149.5
- removed net CLEAN57: JP7.13
- removed net CLEAN570: JP150.1
- removed net CLEAN571: JP150.2
- removed net CLEAN572: JP150.3
- removed net CLEAN573: JP150.4
- removed net CLEAN574: JP150.5
- removed net CLEAN575: JP151.1
- removed net CLEAN576: JP151.2
- removed net CLEAN577: JP151.3
- removed net CLEAN578: JP151.4
- removed net CLEAN579: JP151.5
- removed net CLEAN58: JP7.14
- removed net CLEAN580: JP155.1
- removed net CLEAN581: JP155.2
- removed net CLEAN582: JP155.3
- removed net CLEAN583: JP155.4
- removed net CLEAN584: JP155.5
- removed net CLEAN585: JP156.1
- removed net CLEAN586: JP156.2
- removed net CLEAN587: JP156.3
- removed net CLEAN588: JP156.4
- removed net CLEAN589: JP156.5
- removed net CLEAN59: JP7.15
- removed net CLEAN590: JP157.1
- removed net CLEAN591: JP157.2
- removed net CLEAN592: JP157.3
- removed net CLEAN593: JP157.4
- removed net CLEAN594: JP157.5
- removed net CLEAN595: JP161.1
- removed net CLEAN596: JP161.2
- removed net CLEAN597: JP161.3
- removed net CLEAN598: JP161.4
- removed net CLEAN599: JP161.5
- removed net CLEAN6: JP1.7
- removed net CLEAN60: JP9.1
- removed net CLEAN61: JP9.2
- removed net CLEAN62: JP9.3
- removed net CLEAN63: JP9.4
- removed net CLEAN64: JP9.5
- removed net CLEAN65: JP9.6
- removed net CLEAN66: JP9.7
- removed net CLEAN67: JP9.8
- removed net CLEAN68: JP9.9
- removed net CLEAN69: JP9.10
- removed net CLEAN7: JP1.8
- removed net CLEAN70: JP9.11
- removed net CLEAN71: JP9.12
- removed net CLEAN72: JP9.13
- removed net CLEAN73: JP9.14
- removed net CLEAN74: JP9.15
- removed net CLEAN75: JP11.1
- removed net CLEAN76: JP11.2
- removed net CLEAN77: JP11.3
- removed net CLEAN78: JP11.4
- removed net CLEAN79: JP11.5
- removed net CLEAN8: JP1.9
- removed net CLEAN80: JP11.6
- removed net CLEAN81: JP11.7
- removed net CLEAN82: JP11.8
- removed net CLEAN83: JP11.9
- removed net CLEAN84: JP11.10
- removed net CLEAN85: JP11.11
- removed net CLEAN86: JP11.12
- removed net CLEAN87: JP11.13
- removed net CLEAN88: JP11.14
- removed net CLEAN89: JP11.15
- removed net CLEAN9: JP1.10
- removed net CLEAN90: JP13.1
- removed net CLEAN91: JP13.2
- removed net CLEAN92: JP13.3
- removed net CLEAN93: JP13.4
- removed net CLEAN94: JP13.5
- removed net CLEAN95: JP13.6
- removed net CLEAN96: JP13.7
- removed net CLEAN97: JP13.8
- removed net CLEAN98: JP13.9
- removed net CLEAN99: JP13.10
- new net 0_1438935726: JP132.1, JP21.1
- new net 0_1438935777: JP108.1, JP23.1
- new net 0_1438935827: JP151.1, JP21.15
- new net 0_1438935860: JP144.1, JP23.15
- new net 0_1438935968: JP145.1, JP25.15
- new net 0_1438936000: JP101.1, JP25.1
- new net 0_1438936077: JP27.15, JP67.1
- new net 0_1438936101: JP27.1, JP89.1
- new net 0_1438936131: JP29.1, JP90.1
- new net 0_1438936159: JP29.15, JP55.1
- new net 0_1438936228: JP31.1, JP71.1
- new net 0_1438936248: JP102.1, JP31.15
- new net 0_1438936418: JP103.1, JP33.15
- new net 0_1438936450: JP33.3, JP72.1
- new net 0_1438936529: JP35.8, JP77.1
- new net 0_1438936578: JP35.5, JP73.2
- new net 0_1438936852: JP37.1, JP83.1
- new net 0_1438936878: JP37.13, JP97.1
- new net 0_1438936896: JP39.6, JP85.1
- new net 0_1438936925: JP121.1, JP19.1
- new net 0_1438936947: JP150.1, JP19.15
- new net 0_1438936986: JP149.1, JP17.15
- new net 0_1438937007: JP120.1, JP17.1
- new net 0_1438937040: JP115.1, JP15.1
- new net 0_1438937086: JP15.15, JP156.1
- new net 0_1438937110: JP13.14, JP143.1
- new net 0_1438937129: JP127.1, JP13.1
- new net 0_1438937158: JP11.1, JP125.1
- new net 0_1438937227: JP11.15, JP138.1
- new net 0_1438937250: JP113.1, JP9.15
- new net 0_1438937269: JP42.1, JP9.1
- new net 0_1438937291: JP59.1, JP7.1
- new net 0_1438937314: JP139.1, JP7.13
- new net 0_1438937340: JP5.6, JP61.1
- new net 0_1438937363: JP3.1, JP47.1
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Routing:
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Other:
- board text added: "1"
- board text added: "10"
- board text added: "11"
- board text added: "12"
- board text added: "13"
- board text added: "14"
- board text added: "15"
- board text added: "16"
- board text added: "17"
- board text added: "18"
- board text added: "19"
- board text added: "2"
- board text added: "20"
- board text added: "3"
- board text added: "4"
- board text added: "5"
- board text added: "6"
- board text added: "7"
- board text added: "8"
- board text added: "9"
