File: Eagle/UCirKitBreadboardWithEverything-0812/UCirKitBreadboardWithEverything2.sch (EAGLE design)
At the start: 1200 parts

Commit message: A little error UCirKitBreadboardWithEverthing2 is Bottom part
Parts:
- removed JP1, JP10, JP100, JP101, JP102, JP103, JP104, JP105, JP106, JP107, JP108, JP109, JP11, JP110, JP111, JP112, JP113, JP114, JP115, JP116, JP117, JP118, JP119, JP12, JP120, JP121, JP122, JP123, JP124, JP125, JP126, JP127, JP128, JP129, JP13, JP130, JP131, JP132, JP133, JP134, JP135, JP136, JP137, JP138, JP139, JP14, JP140, JP141, JP142, JP143, JP144, JP145, JP146, JP147, JP148, JP149, JP15, JP150, JP151, JP152, JP153, JP154, JP155, JP156, JP157, JP158, JP159, JP16, JP160, JP161, JP162, JP163, JP164, JP165, JP166, JP167, JP168, JP169, JP17, JP170, JP171, JP172, JP173, JP174, JP175, JP176, JP177, JP178, JP179, JP18, JP180, JP181, JP182, JP183, JP184, JP185, JP186, JP187, JP188, JP189, JP19, JP190, JP191, JP192, JP193, JP194, JP195, JP196, JP197, JP198, JP199, JP2, JP20, JP200, JP201, JP202, JP203, JP204, JP205, JP206, JP207, JP208, JP209, JP21, JP210, JP211, JP212, JP213, JP214, JP215, JP216, JP217, JP218, JP219, JP22, JP220, JP221, JP222, JP223, JP224, JP225, JP226, JP227, JP228, JP229, JP23, JP230, JP231, JP232, JP233, JP234, JP235, JP236, JP237, JP238, JP239, JP24, JP240, JP241, JP242, JP243, JP244, JP245, JP246, JP247, JP248, JP249, JP25, JP250, JP251, JP252, JP253, JP254, JP255, JP256, JP257, JP258, JP259, JP26, JP260, JP261, JP262, JP263, JP264, JP265, JP266, JP267, JP268, JP269, JP27, JP270, JP271, JP272, JP273, JP274, JP275, JP276, JP277, JP278, JP279, JP28, JP280, JP281, JP282, JP283, JP284, JP285, JP286, JP287, JP288, JP289, JP29, JP290, JP291, JP292, JP293, JP294, JP295, JP296, JP297, JP298, JP299, JP3, JP30, JP300, JP31, JP32, JP33, JP34, JP35, JP36, JP37, JP38, JP39, JP4, JP40, JP41, JP42, JP43, JP44, JP45, JP46, JP47, JP48, JP49, JP5, JP50, JP51, JP52, JP53, JP54, JP55, JP56, JP57, JP58, JP59, JP6, JP60, JP61, JP62, JP63, JP64, JP65, JP66, JP67, JP68, JP69, JP7, JP70, JP71, JP72, JP73, JP74, JP75, JP76, JP77, JP78, JP79, JP8, JP80, JP81, JP82, JP83, JP84, JP85, JP86, JP87, JP88, JP89, JP9, JP90, JP91, JP92, JP93, JP94, JP95, JP96, JP97, JP98, JP99: (no value), SparkFun-Connectors:M01PTH_WITHOUT_TEXT

Commit message: UCirKitEverything2Top is OK for Routing, UCirKitEverything2 is not OK. Look for UCirKitEverything2 for Bottom part
Connections:
- new net 0_1439897169: JP301.1, JP841.1
- new net 0_1439897178: JP311.1, JP843.1
- new net 0_1439897188: JP321.1, JP845.1
- new net 0_1439897194: JP310.1, JP781.1
- new net 0_1439897209: JP320.1, JP783.1
- new net 0_1439897217: JP330.1, JP785.1
- new net 0_1439897230: JP340.1, JP787.1
- new net 0_1439897238: JP350.1, JP789.1
- new net 0_1439897247: JP360.1, JP791.1
- new net 0_1439897254: JP370.1, JP793.1
- new net 0_1439897261: JP380.1, JP795.1
- new net 0_1439897267: JP390.1, JP797.1
- new net 0_1439897281: JP600.1, JP839.1
- new net 0_1439897288: JP590.1, JP837.1
- new net 0_1439897294: JP580.1, JP835.1
- new net 0_1439897300: JP591.1, JP899.1
- new net 0_1439897307: JP581.1, JP897.1
- new net 0_1439897312: JP571.1, JP895.1
- new net 0_1439897321: JP561.1, JP893.1
- new net 0_1439897329: JP551.1, JP891.1
- new net 0_1439897335: JP541.1, JP889.1
- new net 0_1439897341: JP531.1, JP887.1
- new net 0_1439897349: JP521.1, JP885.1
- new net 0_1439897354: JP570.1, JP833.1
- new net 0_1439897362: JP560.1, JP831.1
- new net 0_1439897369: JP550.1, JP829.1
- new net 0_1439897383: JP540.1, JP827.1
- new net 0_1439897389: JP530.1, JP825.1
- new net 0_1439897395: JP511.1, JP883.1
- new net 0_1439897401: JP501.1, JP881.1
- new net 0_1439897407: JP491.1, JP879.1
- new net 0_1439897412: JP481.1, JP877.1
- new net 0_1439897418: JP471.1, JP875.1
- new net 0_1439897423: JP461.1, JP873.1
- new net 0_1439897429: JP451.1, JP871.1
- new net 0_1439897436: JP520.1, JP823.1
- new net 0_1439897442: JP510.1, JP821.1
- new net 0_1439897448: JP500.1, JP819.1
- new net 0_1439897454: JP490.1, JP817.1
- new net 0_1439897461: JP480.1, JP815.1
- new net 0_1439897467: JP470.1, JP813.1
- new net 0_1439897473: JP460.1, JP811.1
- new net 0_1439897480: JP450.1, JP809.1
- new net 0_1439897485: JP441.1, JP869.1
- new net 0_1439897491: JP431.1, JP867.1
- new net 0_1439897496: JP421.1, JP865.1
- new net 0_1439897505: JP411.1, JP863.1
- new net 0_1439897514: JP401.1, JP861.1
- new net 0_1439897520: JP440.1, JP807.1
- new net 0_1439897527: JP430.1, JP805.1
- new net 0_1439897534: JP420.1, JP803.1
- new net 0_1439897539: JP410.1, JP801.1
- new net 0_1439897546: JP400.1, JP799.1
- new net 0_1439897614: JP391.1, JP859.1
- new net 0_1439897622: JP381.1, JP857.1
- new net 0_1439897631: JP371.1, JP855.1
- new net 0_1439897637: JP361.1, JP853.1
- new net 0_1439897643: JP351.1, JP851.1
- new net 0_1439897654: JP331.1, JP847.1
- new net 0_1439897660: JP341.1, JP849.1
- new net 0_1439897711: JP593.1, JP651.1
- new net 0_1439897726: JP597.1, JP641.1
- new net 0_1439897746: JP303.1, JP621.1
- new net 0_1439897770: JP307.1, JP601.1
- new net 0_1439897792: JP363.1, JP661.1
- new net 0_1439897815: JP378.1, JP721.1
- new net 0_1439897831: JP473.1, JP695.1
- new net 0_1439897845: JP488.1, JP757.1
- new net 0_1439897966: JP423.1, JP677.1
- new net 0_1439897993: JP428.1, JP737.1
- new net 10_1439897746: JP333.1, JP631.1
- new net 10_1439897770: JP326.1, JP611.1
- new net 10_1439897792: JP375.1, JP671.1
- new net 10_1439897815: JP376.1, JP731.1
- new net 10_1439897831: JP524.1, JP705.1
- new net 10_1439897845: JP537.1, JP767.1
- new net 10_1439897966: JP474.1, JP687.1
- new net 10_1439897993: JP467.1, JP747.1
- new net 11_1439897746: JP343.1, JP632.1
- new net 11_1439897770: JP336.1, JP612.1
- new net 11_1439897792: JP414.1, JP672.1
- new net 11_1439897815: JP417.1, JP732.1
- new net 11_1439897831: JP534.1, JP706.1
- new net 11_1439897845: JP527.1, JP768.1
- new net 11_1439897966: JP435.1, JP688.1
- new net 11_1439897993: JP477.1, JP748.1
- new net 12_1439897746: JP335.1, JP633.1
- new net 12_1439897770: JP348.1, JP613.1
- new net 12_1439897792: JP385.1, JP673.1
- new net 12_1439897815: JP386.1, JP733.1
- new net 12_1439897831: JP544.1, JP707.1
- new net 12_1439897845: JP576.1, JP769.1
- new net 12_1439897966: JP445.1, JP689.1
- new net 12_1439897993: JP446.1, JP749.1
- new net 13_1439897746: JP344.1, JP634.1
- new net 13_1439897770: JP347.1, JP614.1
- new net 13_1439897792: JP395.1, JP674.1
- new net 13_1439897815: JP396.1, JP734.1
- new net 13_1439897831: JP554.1, JP708.1
- new net 13_1439897845: JP566.1, JP770.1
- new net 13_1439897966: JP455.1, JP690.1
- new net 13_1439897993: JP456.1, JP750.1
- new net 14_1439897746: JP345.1, JP635.1
- new net 14_1439897770: JP346.1, JP615.1
- new net 14_1439897792: JP405.1, JP675.1
- new net 14_1439897815: JP406.1, JP735.1
- new net 14_1439897831: JP514.1, JP709.1
- new net 14_1439897845: JP556.1, JP771.1
- new net 14_1439897966: JP465.1, JP691.1
- new net 14_1439897993: JP466.1, JP751.1
- new net 15_1439897746: JP353.1, JP636.1
- new net 15_1439897770: JP358.1, JP616.1
- new net 15_1439897792: JP415.1, JP676.1
- new net 15_1439897815: JP416.1, JP736.1
- new net 15_1439897831: JP504.1, JP710.1
- new net 15_1439897845: JP546.1, JP772.1
- new net 15_1439897966: JP475.1, JP692.1
- new net 15_1439897993: JP476.1, JP752.1
- new net 16_1439897746: JP354.1, JP637.1
- new net 16_1439897770: JP357.1, JP617.1
- new net 16_1439897831: JP545.1, JP711.1
- new net 16_1439897845: JP517.1, JP773.1
- new net 16_1439897966: JP485.1, JP693.1
- new net 16_1439897993: JP486.1, JP753.1
- new net 17_1439897746: JP355.1, JP638.1
- new net 17_1439897770: JP356.1, JP618.1
- new net 17_1439897831: JP555.1, JP712.1
- new net 17_1439897845: JP507.1, JP774.1
- new net 17_1439897966: JP425.1, JP694.1
- new net 17_1439897993: JP496.1, JP754.1
- new net 18_1439897746: JP364.1, JP639.1
- new net 18_1439897770: JP368.1, JP619.1
- new net 18_1439897831: JP565.1, JP713.1
- new net 18_1439897845: JP536.1, JP775.1
- new net 18_1439897993: JP436.1, JP755.1
- new net 19_1439897746: JP365.1, JP640.1
- new net 19_1439897770: JP367.1, JP620.1
- new net 19_1439897831: JP535.1, JP714.1
- new net 19_1439897845: JP497.1, JP776.1
- new net 19_1439897993: JP426.1, JP756.1
- new net 1_1439897169: JP302.1, JP842.1
- new net 1_1439897178: JP312.1, JP844.1
- new net 1_1439897188: JP322.1, JP846.1
- new net 1_1439897194: JP309.1, JP782.1
- new net 1_1439897209: JP319.1, JP784.1
- new net 1_1439897217: JP329.1, JP786.1
- new net 1_1439897230: JP339.1, JP788.1
- new net 1_1439897238: JP349.1, JP790.1
- new net 1_1439897247: JP359.1, JP792.1
- new net 1_1439897254: JP369.1, JP794.1
- new net 1_1439897261: JP379.1, JP796.1
- new net 1_1439897267: JP389.1, JP798.1
- new net 1_1439897281: JP599.1, JP840.1
- new net 1_1439897288: JP589.1, JP838.1
- new net 1_1439897294: JP579.1, JP836.1
- new net 1_1439897300: JP592.1, JP900.1
- new net 1_1439897307: JP582.1, JP898.1
- new net 1_1439897312: JP572.1, JP896.1
- new net 1_1439897321: JP562.1, JP894.1
- new net 1_1439897329: JP552.1, JP892.1
- new net 1_1439897335: JP542.1, JP890.1
- new net 1_1439897341: JP532.1, JP888.1
- new net 1_1439897349: JP522.1, JP886.1
- new net 1_1439897354: JP569.1, JP834.1
- new net 1_1439897362: JP559.1, JP832.1
- new net 1_1439897369: JP549.1, JP830.1
- new net 1_1439897383: JP539.1, JP828.1
- new net 1_1439897389: JP529.1, JP826.1
- new net 1_1439897395: JP512.1, JP884.1
- new net 1_1439897401: JP502.1, JP882.1
- new net 1_1439897407: JP492.1, JP880.1
- new net 1_1439897412: JP482.1, JP878.1
- new net 1_1439897418: JP472.1, JP876.1
- new net 1_1439897423: JP462.1, JP874.1
- new net 1_1439897429: JP452.1, JP872.1
- new net 1_1439897436: JP519.1, JP824.1
- new net 1_1439897442: JP509.1, JP822.1
- new net 1_1439897448: JP499.1, JP820.1
- new net 1_1439897454: JP489.1, JP818.1
- new net 1_1439897461: JP479.1, JP816.1
- new net 1_1439897467: JP469.1, JP814.1
- new net 1_1439897473: JP459.1, JP812.1
- new net 1_1439897480: JP449.1, JP810.1
- new net 1_1439897485: JP442.1, JP870.1
- new net 1_1439897491: JP432.1, JP868.1
- new net 1_1439897496: JP422.1, JP866.1
- new net 1_1439897505: JP412.1, JP864.1
- new net 1_1439897514: JP402.1, JP862.1
- new net 1_1439897520: JP439.1, JP808.1
- new net 1_1439897527: JP429.1, JP806.1
- new net 1_1439897534: JP419.1, JP804.1
- new net 1_1439897539: JP409.1, JP802.1
- new net 1_1439897546: JP399.1, JP800.1
- new net 1_1439897614: JP392.1, JP860.1
- new net 1_1439897622: JP382.1, JP858.1
- new net 1_1439897631: JP372.1, JP856.1
- new net 1_1439897637: JP362.1, JP854.1
- new net 1_1439897643: JP352.1, JP852.1
- new net 1_1439897654: JP332.1, JP848.1
- new net 1_1439897660: JP342.1, JP850.1
- new net 1_1439897711: JP583.1, JP652.1
- new net 1_1439897726: JP598.1, JP642.1
- new net 1_1439897746: JP304.1, JP622.1
- new net 1_1439897770: JP308.1, JP602.1
- new net 1_1439897792: JP373.1, JP662.1
- new net 1_1439897815: JP388.1, JP722.1
- new net 1_1439897831: JP483.1, JP696.1
- new net 1_1439897845: JP498.1, JP758.1
- new net 1_1439897966: JP433.1, JP678.1
- new net 1_1439897993: JP438.1, JP738.1
- new net 20_1439897831: JP525.1, JP715.1
- new net 20_1439897845: JP526.1, JP777.1
- new net 21_1439897831: JP494.1, JP716.1
- new net 21_1439897845: JP487.1, JP778.1
- new net 22_1439897831: JP515.1, JP717.1
- new net 22_1439897845: JP516.1, JP779.1
- new net 23_1439897831: JP505.1, JP718.1
- new net 23_1439897845: JP506.1, JP780.1
- new net 24_1439897831: JP484.1, JP719.1
- new net 25_1439897831: JP495.1, JP720.1
- new net 2_1439897711: JP594.1, JP653.1
- new net 2_1439897726: JP596.1, JP643.1
- new net 2_1439897746: JP313.1, JP623.1
- new net 2_1439897770: JP306.1, JP603.1
- new net 2_1439897792: JP383.1, JP663.1
- new net 2_1439897815: JP377.1, JP723.1
- new net 2_1439897831: JP493.1, JP697.1
- new net 2_1439897845: JP508.1, JP759.1
- new net 2_1439897966: JP443.1, JP679.1
- new net 2_1439897993: JP448.1, JP739.1
- new net 3_1439897711: JP584.1, JP654.1
- new net 3_1439897726: JP588.1, JP644.1
- new net 3_1439897746: JP314.1, JP624.1
- new net 3_1439897770: JP318.1, JP604.1
- new net 3_1439897792: JP374.1, JP664.1
- new net 3_1439897815: JP398.1, JP724.1
- new net 3_1439897831: JP503.1, JP698.1
- new net 3_1439897845: JP518.1, JP760.1
- new net 3_1439897966: JP424.1, JP680.1
- new net 3_1439897993: JP427.1, JP740.1
- new net 4_1439897711: JP573.1, JP655.1
- new net 4_1439897726: JP587.1, JP645.1
- new net 4_1439897746: JP305.1, JP625.1
- new net 4_1439897770: JP317.1, JP605.1
- new net 4_1439897792: JP393.1, JP665.1
- new net 4_1439897815: JP387.1, JP725.1
- new net 4_1439897831: JP513.1, JP699.1
- new net 4_1439897845: JP528.1, JP761.1
- new net 4_1439897966: JP453.1, JP681.1
- new net 4_1439897993: JP458.1, JP741.1
- new net 5_1439897711: JP595.1, JP656.1
- new net 5_1439897726: JP578.1, JP646.1
- new net 5_1439897746: JP315.1, JP626.1
- new net 5_1439897770: JP328.1, JP606.1
- new net 5_1439897792: JP384.1, JP666.1
- new net 5_1439897815: JP366.1, JP726.1
- new net 5_1439897831: JP523.1, JP700.1
- new net 5_1439897845: JP538.1, JP762.1
- new net 5_1439897966: JP434.1, JP682.1
- new net 5_1439897993: JP437.1, JP742.1
- new net 6_1439897711: JP585.1, JP657.1
- new net 6_1439897726: JP577.1, JP647.1
- new net 6_1439897746: JP323.1, JP627.1
- new net 6_1439897770: JP327.1, JP607.1
- new net 6_1439897792: JP403.1, JP667.1
- new net 6_1439897815: JP408.1, JP727.1
- new net 6_1439897831: JP533.1, JP701.1
- new net 6_1439897845: JP548.1, JP763.1
- new net 6_1439897966: JP463.1, JP683.1
- new net 6_1439897993: JP468.1, JP743.1
- new net 7_1439897711: JP574.1, JP658.1
- new net 7_1439897726: JP568.1, JP648.1
- new net 7_1439897746: JP324.1, JP628.1
- new net 7_1439897770: JP338.1, JP608.1
- new net 7_1439897792: JP394.1, JP668.1
- new net 7_1439897815: JP397.1, JP728.1
- new net 7_1439897831: JP543.1, JP702.1
- new net 7_1439897845: JP558.1, JP764.1
- new net 7_1439897966: JP444.1, JP684.1
- new net 7_1439897993: JP447.1, JP744.1
- new net 8_1439897711: JP575.1, JP659.1
- new net 8_1439897726: JP586.1, JP649.1
- new net 8_1439897746: JP325.1, JP629.1
- new net 8_1439897770: JP316.1, JP609.1
- new net 8_1439897792: JP413.1, JP669.1
- new net 8_1439897815: JP418.1, JP729.1
- new net 8_1439897831: JP553.1, JP703.1
- new net 8_1439897845: JP557.1, JP765.1
- new net 8_1439897966: JP454.1, JP685.1
- new net 8_1439897993: JP478.1, JP745.1
- new net 9_1439897711: JP564.1, JP660.1
- new net 9_1439897726: JP567.1, JP650.1
- new net 9_1439897746: JP334.1, JP630.1
- new net 9_1439897770: JP337.1, JP610.1
- new net 9_1439897792: JP404.1, JP670.1
- new net 9_1439897815: JP407.1, JP730.1
- new net 9_1439897831: JP563.1, JP704.1
- new net 9_1439897845: JP547.1, JP766.1
- new net 9_1439897966: JP464.1, JP686.1
- new net 9_1439897993: JP457.1, JP746.1
- new net CLEAN600: JP901.1
- new net CLEAN601: JP902.1
- new net CLEAN602: JP903.1
- new net CLEAN603: JP904.1
- new net CLEAN604: JP905.1
- new net CLEAN605: JP906.1
- new net CLEAN606: JP907.1
- new net CLEAN607: JP908.1
- new net CLEAN608: JP909.1
- new net CLEAN609: JP910.1
- new net CLEAN610: JP911.1
- new net CLEAN611: JP912.1
- new net CLEAN612: JP913.1
- new net CLEAN613: JP914.1
- new net CLEAN614: JP915.1
- new net CLEAN615: JP916.1
- new net CLEAN616: JP917.1
- new net CLEAN617: JP918.1
- new net CLEAN618: JP919.1
- new net CLEAN619: JP920.1
- new net CLEAN620: JP921.1
- new net CLEAN621: JP922.1
- new net CLEAN622: JP923.1
- new net CLEAN623: JP924.1
- new net CLEAN624: JP925.1
- new net CLEAN625: JP926.1
- new net CLEAN626: JP927.1
- new net CLEAN627: JP928.1
- new net CLEAN628: JP929.1
- new net CLEAN629: JP930.1
- new net CLEAN630: JP931.1
- new net CLEAN631: JP932.1
- new net CLEAN632: JP933.1
- new net CLEAN633: JP934.1
- new net CLEAN634: JP935.1
- new net CLEAN635: JP936.1
- new net CLEAN636: JP937.1
- new net CLEAN637: JP938.1
- new net CLEAN638: JP939.1
- new net CLEAN639: JP940.1
- new net CLEAN640: JP941.1
- new net CLEAN641: JP942.1
- new net CLEAN642: JP943.1
- new net CLEAN643: JP944.1
- new net CLEAN644: JP945.1
- new net CLEAN645: JP946.1
- new net CLEAN646: JP947.1
- new net CLEAN647: JP948.1
- new net CLEAN648: JP949.1
- new net CLEAN649: JP950.1
- new net CLEAN650: JP951.1
- new net CLEAN651: JP952.1
- new net CLEAN652: JP953.1
- new net CLEAN653: JP954.1
- new net CLEAN654: JP955.1
- new net CLEAN655: JP956.1
- new net CLEAN656: JP957.1
- new net CLEAN657: JP958.1
- new net CLEAN658: JP959.1
- new net CLEAN659: JP960.1
- new net CLEAN660: JP961.1
- new net CLEAN661: JP962.1
- new net CLEAN662: JP963.1
- new net CLEAN663: JP964.1
- new net CLEAN664: JP965.1
- new net CLEAN665: JP966.1
- new net CLEAN666: JP967.1
- new net CLEAN667: JP968.1
- new net CLEAN668: JP969.1
- new net CLEAN669: JP970.1
- new net CLEAN670: JP971.1
- new net CLEAN671: JP972.1
- new net CLEAN672: JP973.1
- new net CLEAN673: JP974.1
- new net CLEAN674: JP975.1
- new net CLEAN675: JP976.1
- new net CLEAN676: JP977.1
- new net CLEAN677: JP978.1
- new net CLEAN678: JP979.1
- new net CLEAN679: JP980.1
- new net CLEAN680: JP981.1
- new net CLEAN681: JP982.1
- new net CLEAN682: JP983.1
- new net CLEAN683: JP984.1
- new net CLEAN684: JP985.1
- new net CLEAN685: JP986.1
- new net CLEAN686: JP987.1
- new net CLEAN687: JP988.1
- new net CLEAN688: JP989.1
- new net CLEAN689: JP990.1
- new net CLEAN690: JP991.1
- new net CLEAN691: JP992.1
- new net CLEAN692: JP993.1
- new net CLEAN693: JP994.1
- new net CLEAN694: JP995.1
- new net CLEAN695: JP996.1
- new net CLEAN696: JP997.1
- new net CLEAN697: JP998.1
- new net CLEAN698: JP999.1
- new net CLEAN699: JP1000.1
- new net CLEAN700: JP1001.1
- new net CLEAN701: JP1002.1
- new net CLEAN702: JP1003.1
- new net CLEAN703: JP1004.1
- new net CLEAN704: JP1005.1
- new net CLEAN705: JP1006.1
- new net CLEAN706: JP1007.1
- new net CLEAN707: JP1008.1
- new net CLEAN708: JP1009.1
- new net CLEAN709: JP1010.1
- new net CLEAN710: JP1011.1
- new net CLEAN711: JP1012.1
- new net CLEAN712: JP1013.1
- new net CLEAN713: JP1014.1
- new net CLEAN714: JP1015.1
- new net CLEAN715: JP1016.1
- new net CLEAN716: JP1017.1
- new net CLEAN717: JP1018.1
- new net CLEAN718: JP1019.1
- new net CLEAN719: JP1020.1
- new net CLEAN720: JP1021.1
- new net CLEAN721: JP1022.1
- new net CLEAN722: JP1023.1
- new net CLEAN723: JP1024.1
- new net CLEAN724: JP1025.1
- new net CLEAN725: JP1026.1
- new net CLEAN726: JP1027.1
- new net CLEAN727: JP1028.1
- new net CLEAN728: JP1029.1
- new net CLEAN729: JP1030.1
- new net CLEAN730: JP1031.1
- new net CLEAN731: JP1032.1
- new net CLEAN732: JP1033.1
- new net CLEAN733: JP1034.1
- new net CLEAN734: JP1035.1
- new net CLEAN735: JP1036.1
- new net CLEAN736: JP1037.1
- new net CLEAN737: JP1038.1
- new net CLEAN738: JP1039.1
- new net CLEAN739: JP1040.1
- new net CLEAN740: JP1041.1
- new net CLEAN741: JP1042.1
- new net CLEAN742: JP1043.1
- new net CLEAN743: JP1044.1
- new net CLEAN744: JP1045.1
- new net CLEAN745: JP1046.1
- new net CLEAN746: JP1047.1
- new net CLEAN747: JP1048.1
- new net CLEAN748: JP1049.1
- new net CLEAN749: JP1050.1
- new net CLEAN750: JP1051.1
- new net CLEAN751: JP1052.1
- new net CLEAN752: JP1053.1
- new net CLEAN753: JP1054.1
- new net CLEAN754: JP1055.1
- new net CLEAN755: JP1056.1
- new net CLEAN756: JP1057.1
- new net CLEAN757: JP1058.1
- new net CLEAN758: JP1059.1
- new net CLEAN759: JP1060.1
- new net CLEAN760: JP1061.1
- new net CLEAN761: JP1062.1
- new net CLEAN762: JP1063.1
- new net CLEAN763: JP1064.1
- new net CLEAN764: JP1065.1
- new net CLEAN765: JP1066.1
- new net CLEAN766: JP1067.1
- new net CLEAN767: JP1068.1
- new net CLEAN768: JP1069.1
- new net CLEAN769: JP1070.1
- new net CLEAN770: JP1071.1
- new net CLEAN771: JP1072.1
- new net CLEAN772: JP1073.1
- new net CLEAN773: JP1074.1
- new net CLEAN774: JP1075.1
- new net CLEAN775: JP1076.1
- new net CLEAN776: JP1077.1
- new net CLEAN777: JP1078.1
- new net CLEAN778: JP1079.1
- new net CLEAN779: JP1080.1
- new net CLEAN780: JP1081.1
- new net CLEAN781: JP1082.1
- new net CLEAN782: JP1083.1
- new net CLEAN783: JP1084.1
- new net CLEAN784: JP1085.1
- new net CLEAN785: JP1086.1
- new net CLEAN786: JP1087.1
- new net CLEAN787: JP1088.1
- new net CLEAN788: JP1089.1
- new net CLEAN789: JP1090.1
- new net CLEAN790: JP1091.1
- new net CLEAN791: JP1092.1
- new net CLEAN792: JP1093.1
- new net CLEAN793: JP1094.1
- new net CLEAN794: JP1095.1
- new net CLEAN795: JP1096.1
- new net CLEAN796: JP1097.1
- new net CLEAN797: JP1098.1
- new net CLEAN798: JP1099.1
- new net CLEAN799: JP1100.1
- new net CLEAN800: JP1101.1
- new net CLEAN801: JP1102.1
- new net CLEAN802: JP1103.1
- new net CLEAN803: JP1104.1
- new net CLEAN804: JP1105.1
- new net CLEAN805: JP1106.1
- new net CLEAN806: JP1107.1
- new net CLEAN807: JP1108.1
- new net CLEAN808: JP1109.1
- new net CLEAN809: JP1110.1
- new net CLEAN810: JP1111.1
- new net CLEAN811: JP1112.1
- new net CLEAN812: JP1113.1
- new net CLEAN813: JP1114.1
- new net CLEAN814: JP1115.1
- new net CLEAN815: JP1116.1
- new net CLEAN816: JP1117.1
- new net CLEAN817: JP1118.1
- new net CLEAN818: JP1119.1
- new net CLEAN819: JP1120.1
- new net CLEAN820: JP1121.1
- new net CLEAN821: JP1122.1
- new net CLEAN822: JP1123.1
- new net CLEAN823: JP1124.1
- new net CLEAN824: JP1125.1
- new net CLEAN825: JP1126.1
- new net CLEAN826: JP1127.1
- new net CLEAN827: JP1128.1
- new net CLEAN828: JP1129.1
- new net CLEAN829: JP1130.1
- new net CLEAN830: JP1131.1
- new net CLEAN831: JP1132.1
- new net CLEAN832: JP1133.1
- new net CLEAN833: JP1134.1
- new net CLEAN834: JP1135.1
- new net CLEAN835: JP1136.1
- new net CLEAN836: JP1137.1
- new net CLEAN837: JP1138.1
- new net CLEAN838: JP1139.1
- new net CLEAN839: JP1140.1
- new net CLEAN840: JP1141.1
- new net CLEAN841: JP1142.1
- new net CLEAN842: JP1143.1
- new net CLEAN843: JP1144.1
- new net CLEAN844: JP1145.1
- new net CLEAN845: JP1146.1
- new net CLEAN846: JP1147.1
- new net CLEAN847: JP1148.1
- new net CLEAN848: JP1149.1
- new net CLEAN849: JP1150.1
- new net CLEAN850: JP1151.1
- new net CLEAN851: JP1152.1
- new net CLEAN852: JP1153.1
- new net CLEAN853: JP1154.1
- new net CLEAN854: JP1155.1
- new net CLEAN855: JP1156.1
- new net CLEAN856: JP1157.1
- new net CLEAN857: JP1158.1
- new net CLEAN858: JP1159.1
- new net CLEAN859: JP1160.1
- new net CLEAN860: JP1161.1
- new net CLEAN861: JP1162.1
- new net CLEAN862: JP1163.1
- new net CLEAN863: JP1164.1
- new net CLEAN864: JP1165.1
- new net CLEAN865: JP1166.1
- new net CLEAN866: JP1167.1
- new net CLEAN867: JP1168.1
- new net CLEAN868: JP1169.1
- new net CLEAN869: JP1170.1
- new net CLEAN870: JP1171.1
- new net CLEAN871: JP1172.1
- new net CLEAN872: JP1173.1
- new net CLEAN873: JP1174.1
- new net CLEAN874: JP1175.1
- new net CLEAN875: JP1176.1
- new net CLEAN876: JP1177.1
- new net CLEAN877: JP1178.1
- new net CLEAN878: JP1179.1
- new net CLEAN879: JP1180.1
- new net CLEAN880: JP1181.1
- new net CLEAN881: JP1182.1
- new net CLEAN882: JP1183.1
- new net CLEAN883: JP1184.1
- new net CLEAN884: JP1185.1
- new net CLEAN885: JP1186.1
- new net CLEAN886: JP1187.1
- new net CLEAN887: JP1188.1
- new net CLEAN888: JP1189.1
- new net CLEAN889: JP1190.1
- new net CLEAN890: JP1191.1
- new net CLEAN891: JP1192.1
- new net CLEAN892: JP1193.1
- new net CLEAN893: JP1194.1
- new net CLEAN894: JP1195.1
- new net CLEAN895: JP1196.1
- new net CLEAN896: JP1197.1
- new net CLEAN897: JP1198.1
- new net CLEAN898: JP1199.1
- new net CLEAN899: JP1200.1
