File: Eagle/UCirKitUserStudy/UCirKitUserStudy4.sch (EAGLE design)
At the start: 30 parts, among them IC1 74595DIL16-OVAL-PIN, IC2 LM35TO92-EXPANDED-OVAL-PIN

Commit message: UCirKitUserStudy5 has SMD version of resistor, LED, and RGBLED. UCirKitUserStudy4 has oval shape for jumpers.
Parts:
- A0, D10, D11, D12, D13, D3, D4, D5, D6, D7, D8, D9, GND, VCC: device SparkFun-Connectors:M01PTH -> SparkFun-Connectors:M01OVAL_PIN
